File: hardware/PocketLab-Card-routed.kicad_pcb (KiCad board)
At the start: 4 copper layers, 85.6 x 54 mm, 266 parts, among them J1 USB-C DATA/POWER, J2 microSD, J3 EXTERNAL 400uH LF COIL, J4 PROTECTED 1S LiPo 3.7V, J5 30-PIN 2.54mm DUPONT GRID, J8 ER-OLED0.42-1W 72x40 SSD1306B, Q1 AO3400A IR DRIVER, Q2 CSD16406Q3 DISCHARGE, Q3 CSD16406Q3 CHARGE, SW1 RESET, SW2 BOOT, SW3 UP, SW4 DOWN, SW5 MAIN POWER OFF / ON, SW6 PAIR, SW7 SELECT, U1 ESP32-S3-WROOM-1-N8R2, U10 BMI270 (FULL OPTION), U11 BMP390 (FULL OPTION), U12 PCF8563T, U13 TSOP75338WTR 38kHz, U14 BQ29700DSE, U15 TPS2553DBVR 500mA LIMIT, U16 USBLC6-4SC6Y, U17 TPS22919DCKR LF 5V LOAD SWITCH, U18 TCA9534PWR INTERNAL CONTROL, U19 SRV05-4MR6T1G SD ESD, U2 PN5321A3HN/C106, U20 SN74AHCT1G126DBVR RGB LEVEL S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, U21 SN74AHCT125PWR LF 3V3-TO-5V, U22 SN74LVC1G17DBVR LF 5V-TO-3V3, U23 ATECC608C-SSHDA-T, U24 SRV05-4MR6T1G J5 BUS ESD, U25 SRV05-4MR6T1G J5 SPI ESD, U3 E07-900MM10S 855-925MHz, U4 HTRC11001T/03EE,11 125kHz, U5 BQ24074RGTR, U6 TPS63070RNMR 3V3, U7 TPS61023DRLR 5V BOOST, U8 MAX17048G+T10, U9 TCA9535PWR, Y301 27.12MHz crystal (pins 2/4 sh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, Y501 4MHz 5V CMOS OSCILLATOR, Y701 32.768kHz CL=7pF

Commit message: Save RFID and critical routing checkpoint
Parts:
- R102: moved to B.Cu
- moved R102 32.6 mm to (65.7, 36.3), turned to 180 degrees
- moved R201 1.66 mm to (85.5, 47.0), turned to 180 degrees
- moved R202 1.42 mm to (85.5, 49.1), turned to 180 degrees
- moved C404 1.00 mm to (82.8, 66.0), turned to 180 degrees
- moved C314 0.60 mm to (89.2, 47.0)
- moved U16 0.55 mm to (94.0, 50.0)
- moved C106 0.10 mm to (94.2, 49.8)
- turned R405 to 180 degrees
Routing:
- net /NFC_DVDD: track 0.00 -> 67.8 mm
- net /I2C_SCL: track 0.00 -> 57.1 mm, vias 0 -> 3
- net /SPI_MISO: track 0.00 -> 36.8 mm
- net /GPIO44_MCU: track 0.00 -> 29.8 mm, vias 0 -> 2
- net /SPI_MOSI: track 0.00 -> 26.7 mm
- net /SPI_SCK: track 0.00 -> 23.1 mm, vias 0 -> 2
- net /USB_CONN_N: track 21.6 -> 0.00 mm, vias 3 -> 0
- net /USB_CONN_P: track 19.7 -> 0.00 mm, vias 2 -> 0
- net /VSYS: track 16.7 -> 0.00 mm
- net /USB_CC2: track 17.2 -> 4.12 mm, vias 2 -> 0
- net /+5V_RAW: track 11.0 -> 0.00 mm
- net /SUBGHZ_RF_ANT: track 10.3 -> 0.00 mm, vias 1 -> 0
- net /USB_D_P: track 6.47 -> 0.00 mm
- net /USB_D_N: track 5.86 -> 0.00 mm
- net /OLED_VCC: track 0.00 -> 4.63 mm, vias 0 -> 1
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