File: hardware/PocketLab-Card.kicad_sch (KiCad schematic)
At the start: 205 parts, among them J1 USB-C DATA/POWER, J2 microSD, J3 GNSS ANT U.FL, J4 PROTECTED 1S LiPo 3.7V, J5 2x15 2.54mm DUPONT EXPANSION, J6 SUB-GHz ANT U.FL, Q1 AO3400A IR DRIVER, Q2 CSD16406Q3 DISCHARGE, Q3 CSD16406Q3 CHARGE, Q4 AO3400A BUZZER, SW1 RESET, SW2 BOOT, SW3 USER A, SW4 USER B, U1 ESP32-S3-WROOM-1-N8R2, U10 BMI270 (FULL OPTION), U11 BMP390 (FULL OPTION), U12 PCF8563T, U13 TSOP75338WTR 38kHz, U14 BQ29700DSE, U15 TPS2553DBVR 500mA LIMIT, U16 USBLC6-4SC6Y, U17 TPS22919DCKR GNSS LOAD SWITCH, U18 TCA9534PWR INTERNAL CONTROL, U2 PN5321A3HN/C106, U3 E07-900M10S 868MHz, U4 MAX-M10S-00B, U5 BQ24074RGTR, U6 TPS63070RNMR 3V3, U7 TPS61023DRLR 5V BOOST, U8 MAX17048G+T10, U9 TCA9535PWR, Y301 27.12MHz crystal (pins 2/4 sh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, Y701 32.768kHz 12.5pF

Commit message: Publish current PocketLab Card hardware checkpoint
Publishes the current hardware and documentation checkpoint while removing obsolete renders, empty placeholder sheets, generated PCB/autorouter intermediates, and duplicate staging reports. Generated staging artifacts remain reproducible from the checked-in scripts.
Parts:
- removed BZ1: PKMCS0909E, Buzzer_Beeper:Buzzer_Murata_PKMCS0909E, symbol Device:Buzzer
- removed D101: SMF5.0A, Diode_SMD:D_SOD-123F, symbol Device:D_TVS
- removed D501: Low-cap RF ESD, Diode_SMD:D_SOD-523, symbol Device:D_TVS
- removed FB301: 600R@100MHz, Inductor_SMD:L_0805_2012Metric, symbol Device:FerriteBead
- removed J3: GNSS ANT U.FL, Connector_Coaxial:U.FL_Hirose_U.FL-R-SMT-1_Vertical, symbol Connector:Conn_Coaxial
- removed J6: SUB-GHz ANT U.FL, Connector_Coaxial:U.FL_Hirose_U.FL-R-SMT-1_Vertical, symbol Connector:Conn_Coaxial
- removed L501: 27nH high-Q, Inductor_SMD:L_0805_2012Metric, symbol Device:L
- removed Q4: AO3400A BUZZER, Package_TO_SOT_SMD:SOT-23, symbol Transistor_FET:AO3400A
- removed R505: 10R 0.25W, Resistor_SMD:R_0805_2012Metric, symbol Device:R
- removed TP501: GNSS RF TEST, TestPoint:TestPoint_Pad_D1.0mm, symbol Connector:TestPoint
- removed TP601: RGB DOUT, TestPoint:TestPoint_Pad_D1.0mm, symbol Connector:TestPoint
- removed TP701: BMI INT1, TestPoint:TestPoint_Pad_D1.0mm, symbol Connector:TestPoint
- removed TP702: BMP INT, TestPoint:TestPoint_Pad_D1.0mm, symbol Connector:TestPoint
- removed TP703: BMI INT2, TestPoint:TestPoint_Pad_D1.0mm, symbol Connector:TestPoint
- removed U3: E07-900M10S 868MHz, PocketLab_Custom:E07-900M10S, symbol Connector_Generic:Conn_02x11_Odd_Even
- removed U4: MAX-M10S-00B, RF_GPS:ublox_MAX, symbol RF_GPS:MAX-M10S
- added A1: T3-868M SPRING ANTENNA, PocketLab_Custom:T3-868M_Edge_Solder, symbol Device:Antenna
- added C313: 10uF DVDD bulk, Capacitor_SMD:C_0805_2012Metric, symbol Device:C
- added C314: 100nF TVDD, Capacitor_SMD:C_0805_2012Metric, symbol Device:C
- added C315: 4.7uF TVDD bulk, Capacitor_SMD:C_0805_2012Metric, symbol Device:C
- added C316: 100nF PVDD, Capacitor_SMD:C_0805_2012Metric, symbol Device:C
- added C317: 100nF VBAT, Capacitor_SMD:C_0805_2012Metric, symbol Device:C
- added C318: 1nF C0G RX COUPLING, Capacitor_SMD:C_0603_1608Metric, symbol Device:C
- added C403, C404: DNP SUBGHZ MATCH, Capacitor_SMD:C_0805_2012Metric, symbol Device:C
- added C505: 100nF C0G COIL ISOLATION, Capacitor_SMD:C_0805_2012Metric, symbol Device:C
- added C506: 3.9nF C0G LF RESONANCE, Capacitor_SMD:C_0805_2012Metric, symbol Device:C
- added C507: 100pF C0G DNP LF TUNE, Capacitor_SMD:C_0603_1608Metric, symbol Device:C
- added C508: 220pF C0G DNP LF TUNE, Capacitor_SMD:C_0603_1608Metric, symbol Device:C
- added C509: 10pF C0G DNP RX EMI, Capacitor_SMD:C_0603_1608Metric, symbol Device:C
- added C512: 47uF 6.3V LOW-ESR, Capacitor_SMD:C_1210_3225Metric, symbol Device:C
- added C513: 100nF OSC supply, Capacitor_SMD:C_0805_2012Metric, symbol Device:C
- added C515: 100nF AHCT supply, Capacitor_SMD:C_0805_2012Metric, symbol Device:C
- added C516: 100nF LVC supply, Capacitor_SMD:C_0805_2012Metric, symbol Device:C
- added C517: 100nF secure element, Capacitor_SMD:C_0805_2012Metric, symbol Device:C
- added C607, C617: 22uF 10V X5R IR BUFFER, Capacitor_SMD:C_1206_3216Metric, symbol Device:C
- added C608: 100nF IR HF, Capacitor_SMD:C_0805_2012Metric, symbol Device:C
- added C609, C612, C616: 100nF X7R, Capacitor_SMD:C_0805_2012Metric, symbol Device:C
- added C610, C611: 1uF X7R, Capacitor_SMD:C_0805_2012Metric, symbol Device:C
- added C613, C615: 4.7uF X5R, Capacitor_SMD:C_0805_2012Metric, symbol Device:C
- added C614: 2.2uF X7R, Capacitor_SMD:C_0805_2012Metric, symbol Device:C
- added D101: SMF5.0A, Diode_SMD:D_SOD-123F, symbol Device:D_Zener
- added D2, D3: TSAL6200 940nm, PocketLab_Custom:TSAL6200_LayFlat_Inboard, symbol Device:LED
- added J3: EXTERNAL 400uH LF COIL, Connector_PinHeader_2.54mm:PinHeader_1x02_P2.54mm_Vertical, symbol Connector_Generic:Conn_01x02
- added J8: ER-OLED0.42-1W 72x40 SSD1306B, PocketLab_Custom:EastRising_ER-OLED0.42-1W_SolderFPC, symbol Connector_Generic:Conn_01x16
- added R306: 1k VMID BIAS, Resistor_SMD:R_0805_2012Metric, symbol Device:R
- added R406: 100k CS SAFE-HIGH, Resistor_SMD:R_0805_2012Metric, symbol Device:R
- added R506: 100k SAFE-OFF, Resistor_SMD:R_0805_2012Metric, symbol Device:R
- added R509: 10k PAIR pull-up, Resistor_SMD:R_0805_2012Metric, symbol Device:R
- added R610, R611: 39R 0.5W pulse-rated, Resistor_SMD:R_1210_3225Metric, symbol Device:R
- added R722, R723, R724, R725, R726, R727, R728, R729: 220R EXPANSION PROTECTION, Resistor_SMD:R_0603_1608Metric, symbol Device:R
- added R730, R731, R732, R733, R734: 100R, Resistor_SMD:R_0603_1608Metric, symbol Device:R
- added R735: 100k EN pull-down, Resistor_SMD:R_0805_2012Metric, symbol Device:R
- added R736: 10k 1% BOARD TEMP BIAS, Resistor_SMD:R_0603_1608Metric, symbol Device:R
- added RT701: 10k NTC B3950 1%, Resistor_SMD:R_0603_1608Metric, symbol Device:Thermistor
- added SJ1: TS FIXED / CUT FOR EXT NTC, Jumper:SolderJumper-2_P1.3mm_Bridged_RoundedPad1.0x1.5mm, symbol Jumper:SolderJumper_2_Bridged
- added SW5: MAIN POWER OFF / ON, Button_Switch_SMD:SW_SPDT_Shouhan_MSK12C02, symbol Switch:SW_SPDT
- added SW6: PAIR, Button_Switch_SMD:SW_Push_1P1T_NO_CK_KMR2, symbol Switch:SW_Push
- added SW7: SELECT, Button_Switch_SMD:SW_Push_1P1T_NO_CK_KMR2, symbol Switch:SW_Push
- added TP105: POWER VBUS_USB, TestPoint:TestPoint_Pad_D1.0mm, symbol Connector:TestPoint
- added TP106: POWER VBUS_FUSED, TestPoint:TestPoint_Pad_D1.0mm, symbol Connector:TestPoint
- added TP107: POWER VSYS, TestPoint:TestPoint_Pad_D1.0mm, symbol Connector:TestPoint
- added TP108: POWER +3V3, TestPoint:TestPoint_Pad_D1.0mm, symbol Connector:TestPoint
- added TP109: POWER +5V_RAW, TestPoint:TestPoint_Pad_D1.0mm, symbol Connector:TestPoint
- added TP110: POWER +5V_AUX, TestPoint:TestPoint_Pad_D1.0mm, symbol Connector:TestPoint
- added U19: SRV05-4MR6T1G SD ESD, Package_TO_SOT_SMD:SOT-23-6, symbol Power_Protection:SRV05-4
- added U20: SN74AHCT1G126DBVR RGB LEVEL SHIFT, Package_TO_SOT_SMD:SOT-23-5, symbol 74xGxx:74AHCT1G126
- added U21: SN74AHCT125PWR LF 3V3-TO-5V, Package_SO:TSSOP-14_4.4x5mm_P0.65mm, symbol Connector_Generic:Conn_02x07_Odd_Even
- added U22: SN74LVC1G17DBVR LF 5V-TO-3V3, Package_TO_SOT_SMD:SOT-23-5_HandSoldering, symbol 74xGxx:74LVC1G17
- added U23: ATECC608C-SSHDA-T, Package_SO:SOIC-8_3.9x4.9mm_P1.27mm, symbol Security:ATECC608A-SSHDA
- added U24: SRV05-4MR6T1G J5 BUS ESD, Package_TO_SOT_SMD:SOT-23-6, symbol Power_Protection:SRV05-4
- added U25: SRV05-4MR6T1G J5 SPI ESD, Package_TO_SOT_SMD:SOT-23-6, symbol Power_Protection:SRV05-4
- added U3: E07-900MM10S 855-925MHz, PocketLab_Custom:E07-900MM10S, symbol Connector_Generic:Conn_02x10_Odd_Even
- added U4: HTRC11001T/03EE,11 125kHz, Package_SO:SO-14_3.9x8.65mm_P1.27mm, symbol RF_RFID:HTRC11001T
- added Y501: 4MHz 5V CMOS OSCILLATOR, Oscillator:Oscillator_SMD_EuroQuartz_XO32-4Pin_3.2x2.5mm_RotB_HandSoldering, symbol Connector_Generic:Conn_01x04
- AE1: footprint (none) -> PocketLab_Custom:NFC_Loop_35x27mm_4T_TUNE; now left out of the parts list
- C109, C310, C311, C312: DNP (none) -> true; now not fitted
- C302: value 100nF -> 100nF AVDD
- C303: value 4.7uF -> 4.7uF VBAT bulk
- C501: value 100nF -> 100nF HTRC supply
- C502: value 10uF -> 10uF HTRC pulse reservoir
- C503: value 100uF low-leak -> 100nF CEXT; footprint Capacitor_SMD:C_1210_3225Metric -> Capacitor_SMD:C_0805_2012Metric
- C504: value 10nF -> 100nF QGND; footprint Capacitor_SMD:C_0603_1608Metric -> Capacitor_SMD:C_0805_2012Metric
- D1: footprint LED_THT:LED_D5.0mm -> PocketLab_Custom:TSAL6200_LayFlat_Inboard; Assembly (none) -> MANUAL_EDGE_BEND; LCSC (none) -> C55528
- J5: value 2x15 2.54mm DUPONT EXPANSION -> 30-PIN 2.54mm DUPONT GRID; footprint Connector_PinHeader_2.54mm:PinHeader_2x15_P2.54mm_Vertical -> PocketLab_Custom:Dupont_Grid_6x5_P2.54mm
- LED1, LED2, LED3, LED4: value WS2812B-MINI-V3 -> WS2812B-2020; footprint LED_SMD:LED_WS2812B-Mini_PLCC4_3.5x3.5mm -> LED_SMD:LED_WS2812B-2020_PLCC4_2.0x2.0mm; LCSC (none) -> C965555; MPN (none) -> WS2812B-2020; Manufacturer (none) -> Worldsemi
- Q2, Q3: footprint Package_SON:VSON-8_3.3x3.3mm_P0.65mm_NexFET -> PocketLab_Custom:CSD16406Q3_VSON-8_3.3x3.3mm_P0.65mm_JLC
- R302: value 10k -> 10k RESET default asserted
- R305: value 1k RX TAP -> 2.7k RX TAP
- R405: value 0R ANT SELECT -> 0R SUBGHZ MATCH
- R502: value 10k -> 47R 0.5W ANTENNA CURRENT LIMIT; footprint Resistor_SMD:R_0805_2012Metric -> Resistor_SMD:R_1210_3225Metric
- R503: value 100R -> 1k LF EMI RETURN
- R504: value 0R RF -> 150k 1% RX DIVIDER
- R601: value 39R 1W pulse-rated -> 39R 0.5W pulse-rated; footprint Resistor_SMD:R_2512_6332Metric -> Resistor_SMD:R_1210_3225Metric
- R605: value 330R -> 68R; footprint Resistor_SMD:R_0805_2012Metric -> Resistor_SMD:R_0603_1608Metric
- R606: value 100R -> 100R PAIR GPIO PROTECTION; footprint Resistor_SMD:R_0805_2012Metric -> Resistor_SMD:R_0603_1608Metric
- R607: value 100k -> 10k; footprint Resistor_SMD:R_0805_2012Metric -> Resistor_SMD:R_0603_1608Metric
- R608, R609, R710, R711, R712, R713, R715, R716, R717, R718, R719, R720, R721: footprint Resistor_SMD:R_0805_2012Metric -> Resistor_SMD:R_0603_1608Metric
- R701, R702: value 4.7k -> 3.3k
- R714: value 100R -> 100R BOARD TEMP PROBE; footprint Resistor_SMD:R_0805_2012Metric -> Resistor_SMD:R_0603_1608Metric
- SW1, SW2: footprint Button_Switch_SMD:SW_SPST_TL3305A -> Button_Switch_SMD:SW_Push_1P1T_NO_CK_KMR2; LCSC (none) -> C72443; MPN (none) -> KMR221GLFS; Manufacturer (none) -> C&K
- SW3: value USER A -> UP; footprint Button_Switch_SMD:SW_SPST_TL3305A -> Button_Switch_SMD:SW_Push_1P1T_NO_CK_KMR2; LCSC (none) -> C72443; MPN (none) -> KMR221GLFS; Manufacturer (none) -> C&K
- SW4: value USER B -> DOWN; footprint Button_Switch_SMD:SW_SPST_TL3305A -> Button_Switch_SMD:SW_Push_1P1T_NO_CK_KMR2; LCSC (none) -> C72443; MPN (none) -> KMR221GLFS; Manufacturer (none) -> C&K
- TP101, TP102, TP103, TP104, TP201, TP202, TP203, TP301: now left out of the parts list
- TP502: value LNA ENABLE -> LF ANTENNA TAP - HIGH VOLTAGE; now left out of the parts list
- U1: footprint RF_Module:ESP32-S3-WROOM-1 -> PocketLab_Card:ESP32-S3-WROOM-1_PhysicalCourtyard
- U17: value TPS22919DCKR GNSS LOAD SWITCH -> TPS22919DCKR LF 5V LOAD SWITCH; LCSC (none) -> C2149796
- Y701: value 32.768kHz 12.5pF -> 32.768kHz CL=7pF; MPN (none) -> ABS07-32.768KHZ-7-T; Manufacturer (none) -> Abracon
Connections:
- net GNSS_RF is gone; now on net LF_TAP: R504.1
- net NFC_AVDD is gone; now on net NFC_DVDD: C302.1, U2.8 (AVDD)
- net +3V3: now also R607.2, C316.1, C317.1, C512.1, C516.1, C517.1, C612.1, C613.1, J8.5 (Pin_5), J8.7 (Pin_7), J8.8 (Pin_8), R406.2, R509.2, R736.1, TP108.1, U19.5 (VP), U22.5 (VCC), U23.8 (VCC), U24.5 (VP), U25.5 (VP), U3.1 (Pin_1); no longer C603.1, C604.1, C605.1, C606.1, LED1.1 (VDD), LED2.1 (VDD), LED3.1 (VDD), LED4.1 (VDD), R302.2, U17.1 (Pin_1), U2.5 (TVDD)
- net +5V_AUX: now also TP110.1
- net +5V_RAW: now also C603.1, C604.1, C605.1, C606.1, LED1.1 (VDD), LED2.1 (VDD), LED3.1 (VDD), LED4.1 (VDD), U17.1 (Pin_1), C607.1, C608.1, C609.1, C617.1, R610.1, R611.1, TP109.1, U20.5 (VCC)
- net BOOST5_EN: now also U20.1
- net CHG_TS: now also J5.28 (Pin_28), SJ1.1 (A); no longer R108.1
- net ESP_EN: now also J8.10 (Pin_10)
- net EX0: now also R722.2; no longer U9.13 (P10)
- net EX1: now also R723.2; no longer U9.14 (P11)
- net EX2: now also R724.2; no longer U9.15 (P12)
- net EX3: now also R725.2; no longer U9.16 (P13)
- net EX4: now also R726.2; no longer U9.17 (P14)
- net EX5: now also R727.2; no longer U9.18 (P15)
- net EX6: now also R728.2; no longer U9.19 (P16)
- net EX7: now also R729.2; no longer U9.20 (P17)
- net GND: now also R302.2, R503.2, C313.2, C314.2, C315.2, C316.2, C317.2, C403.2, C404.2, C512.2, C513.2, C515.2, C516.2, C517.2, C607.2, C608.2, C609.2, C612.2, C613.2, C614.2, C615.2, C616.2, C617.2, D101.2 (A), J8.11 (Pin_11), J8.6 (Pin_6), J8.9 (Pin_9), R506.2, R735.2, RT701.2, SW5.1 (A), SW6.2, SW7.2, U19.2 (VN), U20.3 (GND), U21.1 (Pin_1), U21.12 (Pin_12), U21.4 (Pin_4), U21.7 (Pin_7), U21.9 (Pin_9), U22.3 (GND), U23.4 (GND), U24.2 (VN), U25.2 (VN), U3.16 (Pin_16), U3.2 (Pin_2), U3.7 (Pin_7), U4.1 (VSS), U4.5 (MODE), Y501.2 (Pin_2); no longer J5.28 (Pin_28), R607.2
- net I2C_SCL: now also J8.12 (Pin_12), R731.1, U23.6 (SCL); no longer J5.24 (Pin_24)
- net I2C_SDA: now also J8.13 (Pin_13), J8.14 (Pin_14), R730.1, U23.5 (SDA); no longer J5.23 (Pin_23)
- net IR_LED_K: now also D2.1 (K), D3.1 (K)
- net NFC_DVDD: now also U2.5 (TVDD), C313.1, C314.1, C315.1
- net NFC_RX: now also C318.2, R306.2; no longer R305.2
- net NFC_VMID: now also R306.1
- net RGB_DATA: now also U20.2; no longer R605.1
- net SD_CS_DEV: now also U19.1 (IO1)
- net SD_MISO: now also U19.6 (IO4)
- net SD_MOSI: now also U19.3 (IO2)
- net SD_SCK: now also U19.4 (IO3)
- net SPI_MISO: now also R734.1; no longer J5.27 (Pin_27)
- net SPI_MOSI: now also R733.1; no longer J5.26 (Pin_26)
- net SPI_SCK: now also R732.1; no longer J5.25 (Pin_25)
- net SUBGHZ_GDO0: now also U3.18 (Pin_18)
- net SUBGHZ_GDO2: now also U3.20 (Pin_20)
- net SUB_CS_N: now also R406.1, U3.14 (Pin_14)
- net SUB_MISO: now also U3.12 (Pin_12)
- net SUB_MOSI: now also U3.13 (Pin_13)
- net SUB_SCK: now also U3.15 (Pin_15)
- net U6_PS_SYNC: now also U6.14 (Pin_14), R735.1, SW5.2 (B); no longer R116.2
- net VBUS_FUSED: now also D101.1 (K), TP106.1
- net VBUS_USB: now also TP105.1
- net VSYS: now also TP107.1; no longer U6.14 (Pin_14)
- net BMP_INT: no longer names the net of U11.7 (Pin_7)
- net BMP_INT: no longer U9.11 (P07)
- net BUZZER_GATE renamed PAIR_N
- net PAIR_N: now also R509.1, SW6.1; no longer R607.1
- net BUZZER_PWM renamed GPIO38_MCU
- net GNSS_3V3 renamed LF_5V
- net LF_5V: now also C513.1, C515.1, U21.10 (Pin_10), U21.13 (Pin_13), U21.14 (Pin_14), U4.3 (VDD), Y501.1 (Pin_1), Y501.4 (Pin_4); no longer R502.2, R503.1
- net GNSS_ANT_FEED renamed LF_RX
- net LF_RX: now also C509.1, U4.14 (RX)
- net GNSS_BACKUP renamed LF_CEXT
- net LF_CEXT: now also U4.12 (CEXT); no longer R503.2
- net GNSS_BIAS renamed LF_QGND
- net LF_QGND: now also C509.2, U4.13 (QGND)
- net GNSS_LNA_EN renamed LF_TAP
- net LF_TAP: now also R502.2, C506.1, C507.1, C508.1
- net GNSS_POWER_EN renamed LF_RFID_EN
- net LF_RFID_EN: now also R506.1
- net GNSS_QOD renamed LF_QOD
- net GNSS_RESET_N renamed LF_ANT_B
- net LF_ANT_B: now also J3.2 (Pin_2)
- net GNSS_RX_FROM_MODULE renamed LF_DOUT_3V3
- net LF_DOUT_3V3: now also U22.4
- net GNSS_TIMEPULSE renamed LF_SCLK_3V3
- net LF_SCLK_3V3: now also U21.2 (Pin_2)
- net GNSS_TX_TO_MODULE renamed LF_DIN_3V3
- net LF_DIN_3V3: now also U21.5 (Pin_5)
- net GPIO9 renamed BOARD_TEMP_HDR
- net GPIO9_MCU renamed BOARD_TEMP_ADC
- net BOARD_TEMP_ADC: now also R736.2, RT701.1
- net IR_LED_A renamed IR_LED_A1
- net RGB_DOUT4: no longer names the net of LED4.2 (DOUT)
- net SUBGHZ_ANT renamed SUBGHZ_RF_ANT
- net SUBGHZ_RF_ANT: now also A1.1 (A), C404.1
- net SUBGHZ_RF renamed SUBGHZ_RF_MOD
- net SUBGHZ_RF_MOD: now also C403.1, U3.6 (Pin_6)
- net USB_DM_CONN renamed USB_CONN_N
- net USB_DP_CONN renamed USB_CONN_P
- new net CHG_TS_FIXED: R108.1, SJ1.2 (B)
- new net EX0_INT: R722.1, U9.13 (P10)
- new net EX1_INT: R723.1, U9.14 (P11)
- new net EX2_INT: R724.1, U9.15 (P12)
- new net EX3_INT: R725.1, U9.16 (P13)
- new net EX4_INT: R726.1, U9.17 (P14)
- new net EX5_INT: R727.1, U9.18 (P15)
- new net EX6_INT: R728.1, U9.19 (P16)
- new net EX7_INT: R729.1, U9.20 (P17)
- new net I2C_SCL_HDR: J5.24 (Pin_24), R731.2, U24.3 (IO2)
- new net I2C_SDA_HDR: J5.23 (Pin_23), R730.2, U24.1 (IO1)
- new net IR_LED_A2: D2.2 (A), R610.2
- new net IR_LED_A3: D3.2 (A), R611.2
- new net LF_ANT_A: C505.2, J3.1 (Pin_1), R503.1
- new net LF_CLK_4M: U4.6 (XTAL1), Y501.3 (Pin_3)
- new net LF_DIN_5V: U21.6 (Pin_6), U4.9 (DIN)
- new net LF_DOUT_5V: U22.2, U4.10 (DOUT)
- new net LF_SCLK_5V: U21.3 (Pin_3), U4.8 (SCLK)
- new net LF_TX1: C505.1, U4.4 (TX1)
- new net LF_TX2: C506.2, C507.2, C508.2, U4.2 (TX2)
- new net NFC_RX_AC: C318.1, R305.2
- new net OLED_C1N: C611.2, J8.4 (Pin_4)
- new net OLED_C1P: C611.1, J8.3 (Pin_3)
- new net OLED_C2N: C610.2, J8.2 (Pin_2)
- new net OLED_C2P: C610.1, J8.1 (Pin_1)
- new net OLED_VCC: C615.1, C616.1, J8.16 (Pin_16)
- new net OLED_VCOMH: C614.1, J8.15 (Pin_15)
- new net PWR_SW_ON: R116.2, SW5.3 (C)
- new net RGB_BUF_5V: R605.1, U20.4
- new net SPI_MISO_HDR: J5.27 (Pin_27), R734.2, U25.1 (IO1)
- new net SPI_MOSI_HDR: J5.26 (Pin_26), R733.2, U25.3 (IO2)
- new net SPI_SCK_HDR: J5.25 (Pin_25), R732.2, U25.4 (IO3)
- new net USER_BUTTON_SELECT_N: R607.1, SW7.1, U9.11 (P07)
- no-connect marks 36 -> 48
Other:
- note added: "05 LF RFID / SECURITY / MICROSD"
- note added: "06 IR / RGB / BUTTONS / OLED"
- note removed: "05 GNSS / ANTENNA / MICROSD"
- note removed: "06 IR / RGB / BUTTONS / BUZZER"
