File: hardware/PocketLab-Card.kicad_sch (KiCad schematic)
At the start: 0 parts

Commit message: Save complete schematic and firmware checkpoint
Parts:
- added AE1: PCB NFC LOOP - TUNE ON V1, symbol Device:Antenna_Loop
- added BZ1: PKMCS0909E, Buzzer_Beeper:Buzzer_Murata_PKMCS0909E, symbol Device:Buzzer
- added C101: 4.7nF 1kV, Capacitor_SMD:C_0805_2012Metric, symbol Device:C
- added C102, C106, C107, C118, C120, C121, C122, C203, C301, C302, C304, C305, C401, C501, C510, C601, C603, C604, C605, C606, C701, C706, C707: 100nF, Capacitor_SMD:C_0805_2012Metric, symbol Device:C
- added C103, C105: 4.7uF 10V, Capacitor_SMD:C_0805_2012Metric, symbol Device:C
- added C104: 22uF 10V, Capacitor_SMD:C_0805_2012Metric, symbol Device:C
- added C108, C114, C117, C119, C202, C502, C511: 10uF, Capacitor_SMD:C_0805_2012Metric, symbol Device:C
- added C109: 10uF DNP - populate only after VSYS stability test, Capacitor_SMD:C_0805_2012Metric, symbol Device:C
- added C110, C111, C112, C115, C116: 22uF, Capacitor_SMD:C_0805_2012Metric, symbol Device:C
- added C113, C308, C309: 220pF C0G, Capacitor_SMD:C_0603_1608Metric, symbol Device:C
- added C123, C124: 10uF 25V X5R HF, Capacitor_SMD:C_0603_1608Metric, symbol Device:C
- added C201: 1uF, Capacitor_SMD:C_0805_2012Metric, symbol Device:C
- added C303, C402, C602: 4.7uF, Capacitor_SMD:C_0805_2012Metric, symbol Device:C
- added C306, C307: 22pF C0G, Capacitor_SMD:C_0603_1608Metric, symbol Device:C
- added C310, C311, C312: DNP MATCH, Capacitor_SMD:C_0603_1608Metric, symbol Device:C
- added C503: 100uF low-leak, Capacitor_SMD:C_1210_3225Metric, symbol Device:C
- added C504: 10nF, Capacitor_SMD:C_0603_1608Metric, symbol Device:C
- added C702, C703, C704, C705: 100nF, Capacitor_SMD:C_0603_1608Metric, symbol Device:C
- added D1: TSAL6200 940nm, LED_THT:LED_D5.0mm, symbol Device:LED
- added D101: SMF5.0A, Diode_SMD:D_SOD-123F, symbol Device:D_TVS
- added D501: Low-cap RF ESD, Diode_SMD:D_SOD-523, symbol Device:D_TVS
- added F1: Littelfuse 1206L075/13.2, Fuse:Fuse_1206_3216Metric, symbol Device:Polyfuse
- added FB301: 600R@100MHz, Inductor_SMD:L_0805_2012Metric, symbol Device:FerriteBead
- added J1: USB-C DATA/POWER, Connector_USB:USB_C_Receptacle_HRO_TYPE-C-31-M-12, symbol Connector:USB_C_Receptacle_USB2.0_14P
- added J2: microSD, Connector_Card:microSD_HC_Molex_104031-0811, symbol Connector:Micro_SD_Card_Det2
- added J3: GNSS ANT U.FL, Connector_Coaxial:U.FL_Hirose_U.FL-R-SMT-1_Vertical, symbol Connector:Conn_Coaxial
- added J4: PROTECTED 1S LiPo 3.7V, Connector_JST:JST_PH_S2B-PH-SM4-TB_1x02-1MP_P2.00mm_Horizontal, symbol Connector_Generic:Conn_01x02
- added J5: 2x15 2.54mm DUPONT EXPANSION, Connector_PinHeader_2.54mm:PinHeader_2x15_P2.54mm_Vertical, symbol Connector_Generic:Conn_02x15_Odd_Even
- added J6: SUB-GHz ANT U.FL, Connector_Coaxial:U.FL_Hirose_U.FL-R-SMT-1_Vertical, symbol Connector:Conn_Coaxial
- added L301, L302: 560nH C0G/Q, Inductor_SMD:L_0805_2012Metric, symbol Device:L
- added L501: 27nH high-Q, Inductor_SMD:L_0805_2012Metric, symbol Device:L
- added L6: 1.5uH XFL4020-152ME, PocketLab_Custom:Coilcraft_XFL4020, symbol Device:L
- added L7: 1uH HBME042A, PocketLab_Custom:Cyntec_HBME042A-1R0MS, symbol Device:L
- added LED1, LED2, LED3, LED4: WS2812B-MINI-V3, LED_SMD:LED_WS2812B-Mini_PLCC4_3.5x3.5mm, symbol LED:WS2812B
- added Q1: AO3400A IR DRIVER, Package_TO_SOT_SMD:SOT-23, symbol Transistor_FET:AO3400A
- added Q2: CSD16406Q3 DISCHARGE, Package_SON:VSON-8_3.3x3.3mm_P0.65mm_NexFET, symbol Connector_Generic:Conn_01x05
- added Q3: CSD16406Q3 CHARGE, Package_SON:VSON-8_3.3x3.3mm_P0.65mm_NexFET, symbol Connector_Generic:Conn_01x05
- added Q4: AO3400A BUZZER, Package_TO_SOT_SMD:SOT-23, symbol Transistor_FET:AO3400A
- added R101, R102: 5.1k 1%, Resistor_SMD:R_0805_2012Metric, symbol Device:R
- added R103: 1M, Resistor_SMD:R_0805_2012Metric, symbol Device:R
- added R104, R605: 330R, Resistor_SMD:R_0805_2012Metric, symbol Device:R
- added R105: 2.2k, Resistor_SMD:R_0805_2012Metric, symbol Device:R
- added R106, R107: 5.1M, Resistor_SMD:R_0805_2012Metric, symbol Device:R
- added R108: 10k TS fixed, Resistor_SMD:R_0805_2012Metric, symbol Device:R
- added R109, R110, R115, R122, R124, R126, R127, R128, R603, R607: 100k, Resistor_SMD:R_0805_2012Metric, symbol Device:R
- added R111: 3.48k 1%, Resistor_SMD:R_0805_2012Metric, symbol Device:R
- added R112: 3.01k 1%, Resistor_SMD:R_0805_2012Metric, symbol Device:R
- added R113: 1.78k 1%, Resistor_SMD:R_0805_2012Metric, symbol Device:R
- added R114: 68.1k 1%, Resistor_SMD:R_0805_2012Metric, symbol Device:R
- added R116, R119, R125, R203, R204, R301, R302, R502, R519, R608, R609, R703: 10k, Resistor_SMD:R_0805_2012Metric, symbol Device:R
- added R117: 470k 1%, Resistor_SMD:R_0805_2012Metric, symbol Device:R
- added R118: 150k 1%, Resistor_SMD:R_0805_2012Metric, symbol Device:R
- added R120: 732k 1%, Resistor_SMD:R_0805_2012Metric, symbol Device:R
- added R121: 100k 1%, Resistor_SMD:R_0805_2012Metric, symbol Device:R
- added R123: 60.4k 1%, Resistor_SMD:R_0805_2012Metric, symbol Device:R
- added R201, R202, R401, R402, R403, R404, R510, R511, R512, R513: 22R, Resistor_SMD:R_0805_2012Metric, symbol Device:R
- added R303, R304: 0R MATCH, Resistor_SMD:R_0805_2012Metric, symbol Device:R
- added R305: 1k RX TAP, Resistor_SMD:R_0805_2012Metric, symbol Device:R
- added R405: 0R ANT SELECT, Resistor_SMD:R_0805_2012Metric, symbol Device:R
- added R501: 100R QOD discharge, Resistor_SMD:R_0805_2012Metric, symbol Device:R
- added R503, R602, R604, R606, R710, R711, R712, R713, R714, R715, R716, R717, R718, R719, R720, R721: 100R, Resistor_SMD:R_0805_2012Metric, symbol Device:R
- added R504: 0R RF, Resistor_SMD:R_0805_2012Metric, symbol Device:R
- added R505: 10R 0.25W, Resistor_SMD:R_0805_2012Metric, symbol Device:R
- added R514, R515, R516, R517, R518: 47k, Resistor_SMD:R_0805_2012Metric, symbol Device:R
- added R601: 39R 1W pulse-rated, Resistor_SMD:R_2512_6332Metric, symbol Device:R
- added R701, R702: 4.7k, Resistor_SMD:R_0805_2012Metric, symbol Device:R
- added SW1: RESET, Button_Switch_SMD:SW_SPST_TL3305A, symbol Switch:SW_Push
- added SW2: BOOT, Button_Switch_SMD:SW_SPST_TL3305A, symbol Switch:SW_Push
- added SW3: USER A, Button_Switch_SMD:SW_SPST_TL3305A, symbol Switch:SW_Push
- added SW4: USER B, Button_Switch_SMD:SW_SPST_TL3305A, symbol Switch:SW_Push
- added TP101: BATTERY CELL_POS, TestPoint:TestPoint_Pad_D1.0mm, symbol Connector:TestPoint
- added TP102: BATTERY CELL_NEG, TestPoint:TestPoint_Pad_D1.0mm, symbol Connector:TestPoint
- added TP103: BATTERY BAT_FET_MID, TestPoint:TestPoint_Pad_D1.0mm, symbol Connector:TestPoint
- added TP104: BATTERY GND, TestPoint:TestPoint_Pad_D1.0mm, symbol Connector:TestPoint
- added TP201: JTAG_STRAP_TP, TestPoint:TestPoint_Pad_D1.0mm, symbol Connector:TestPoint
- added TP202: STRAP_BOOT_TP, TestPoint:TestPoint_Pad_D1.0mm, symbol Connector:TestPoint
- added TP203: STRAP_VDD_SPI_TP, TestPoint:TestPoint_Pad_D1.0mm, symbol Connector:TestPoint
- added TP301: NFC_LOADMOD TEST, TestPoint:TestPoint_Pad_D1.0mm, symbol Connector:TestPoint
- added TP501: GNSS RF TEST, TestPoint:TestPoint_Pad_D1.0mm, symbol Connector:TestPoint
- added TP502: LNA ENABLE, TestPoint:TestPoint_Pad_D1.0mm, symbol Connector:TestPoint
- added TP601: RGB DOUT, TestPoint:TestPoint_Pad_D1.0mm, symbol Connector:TestPoint
- added TP701: BMI INT1, TestPoint:TestPoint_Pad_D1.0mm, symbol Connector:TestPoint
- added TP702: BMP INT, TestPoint:TestPoint_Pad_D1.0mm, symbol Connector:TestPoint
- added TP703: BMI INT2, TestPoint:TestPoint_Pad_D1.0mm, symbol Connector:TestPoint
- added U1: ESP32-S3-WROOM-1-N8R2, RF_Module:ESP32-S3-WROOM-1, symbol RF_Module:ESP32-S3-WROOM-1
- added U10: BMI270 (FULL OPTION), Package_LGA:Bosch_LGA-14_3x2.5mm_P0.5mm, symbol Connector_Generic:Conn_02x07_Odd_Even
- added U11: BMP390 (FULL OPTION), PocketLab_Custom:BMP390_LGA-10_2x2mm, symbol Connector_Generic:Conn_02x05_Odd_Even
- added U12: PCF8563T, Package_SO:SOIC-8_3.9x4.9mm_P1.27mm, symbol Timer_RTC:PCF8563T
- added U13: TSOP75338WTR 38kHz, PocketLab_Custom:TSOP75338WTR_HeimdallW_SideView, symbol Connector_Generic:Conn_01x04
- added U14: BQ29700DSE, Package_SON:WSON-6_1.5x1.5mm_P0.5mm, symbol Battery_Management:BQ297xy
- added U15: TPS2553DBVR 500mA LIMIT, Package_TO_SOT_SMD:SOT-23-6, symbol Connector_Generic:Conn_01x06
- added U16: USBLC6-4SC6Y, Package_TO_SOT_SMD:SOT-23-6, symbol Power_Protection:USBLC6-4SC6
- added U17: TPS22919DCKR GNSS LOAD SWITCH, Package_TO_SOT_SMD:SOT-363_SC-70-6, symbol Connector_Generic:Conn_01x06
- added U18: TCA9534PWR INTERNAL CONTROL, Package_SO:TSSOP-16_4.4x5mm_P0.65mm, symbol Interface_Expansion:TCA9534
- added U2: PN5321A3HN/C106, Package_DFN_QFN:HVQFN-40-1EP_6x6mm_P0.5mm_EP4.1x4.1mm, symbol RF_NFC:PN5321A3HN_C1xx
- added U3: E07-900M10S 868MHz, PocketLab_Custom:E07-900M10S, symbol Connector_Generic:Conn_02x11_Odd_Even
- added U4: MAX-M10S-00B, RF_GPS:ublox_MAX, symbol RF_GPS:MAX-M10S
- added U5: BQ24074RGTR, Package_DFN_QFN:VQFN-16-1EP_3x3mm_P0.5mm_EP1.6x1.6mm_ThermalVias, symbol Battery_Management:BQ24074RGT
- added U6: TPS63070RNMR 3V3, PocketLab_Custom:TPS63070_RNM0015A, symbol Connector_Generic:Conn_01x15
- added U7: TPS61023DRLR 5V BOOST, Package_TO_SOT_SMD:SOT-563, symbol Connector_Generic:Conn_01x06
- added U8: MAX17048G+T10, Package_DFN_QFN:TDFN-8-1EP_2x2mm_P0.5mm_EP0.8x1.2mm, symbol Connector_Generic:Conn_01x09
- added U9: TCA9535PWR, Package_SO:TSSOP-24_4.4x7.8mm_P0.65mm, symbol Interface_Expansion:TCA9535DBR
- added Y301: 27.12MHz crystal (pins 2/4 shield), Crystal:Crystal_SMD_3225-4Pin_3.2x2.5mm, symbol Connector_Generic:Conn_01x04
- added Y701: 32.768kHz 12.5pF, Crystal:Crystal_SMD_3215-2Pin_3.2x1.5mm, symbol Device:Crystal
Connections:
- new net +3V3: BZ1.1 (+), C110.1, C111.1, C112.1, C124.1, C202.1, C203.1, C303.1, C401.1, C402.1, C510.1, C511.1, C603.1, C604.1, C605.1, C606.1, C701.1, C702.1, C703.1, C704.1, C705.1, C706.1, C707.1, FB301.1, J2.4 (VDD), J5.1 (Pin_1), LED1.1 (VDD), LED2.1 (VDD), LED3.1 (VDD), LED4.1 (VDD), R109.2, R110.2, R117.1, R119.2, R124.2, R125.2, R203.2, R204.2, R302.2, R514.2, R515.2, R516.2, R517.2, R518.2, R519.2, R604.1, R608.2, R609.2, R701.2, R702.2, R703.2, U1.2 (3V3), U10.12 (Pin_12), U10.5 (Pin_5), U10.8 (Pin_8), U11.1 (Pin_1), U11.10 (Pin_10), U11.6 (Pin_6), U12.8 (VDD), U17.1 (Pin_1), U18.1 (A0), U18.16 (VDD), U2.23 (PVDD), U2.40 (VBAT), U2.5 (TVDD), U3.9 (Pin_9), U6.7 (Pin_7), U6.8 (Pin_8), U9.24 (VCC)
- new net +5V_AUX: C118.1, C119.1, J5.29 (Pin_29), U15.6 (Pin_6)
- new net +5V_RAW: C113.1, C115.1, C116.1, C117.1, R120.1, R601.1, U15.1 (Pin_1), U7.6 (Pin_6)
- new net AUX5_EN: R127.1, U15.3 (Pin_3), U18.6 (P2)
- new net AUX5_FAULT_N: R124.1, U15.4 (Pin_4), U9.7 (P03)
- new net BAT_COUT: Q3.4 (Pin_4), R107.1, U14.2 (Cout)
- new net BAT_DOUT: Q2.4 (Pin_4), R106.1, U14.3 (Dout)
- new net BAT_FET_MID: Q2.5 (Pin_5), Q3.5 (Pin_5), TP103.1
- new net BAT_SENSE: C102.1, R104.2, U14.5 (BAT)
- new net BAT_VMINUS: R105.1, U14.6 (V-)
- new net BMI_INT1: TP701.1, U10.4 (Pin_4), U9.9 (P05)
- new net BMI_INT2: TP703.1, U10.9 (Pin_9), U9.10 (P06)
- new net BMP_INT: TP702.1, U11.7 (Pin_7), U9.11 (P07)
- new net BOOST5_EN: R122.1, U18.10 (P5), U7.2 (Pin_2)
- new net BOOT_N: R204.1, SW2.1, U1.27 (IO0)
- new net BQ_EN1: R115.1, U18.4 (P0), U5.6 (EN1)
- new net BQ_EN2: R128.1, U5.5 (EN2)
- new net BUZZER_GATE: Q4.1 (G), R606.2, R607.1
- new net BUZZER_NEG: BZ1.2 (-), Q4.3 (D)
- new net BUZZER_PWM: R606.1, U1.31 (IO38)
- new net CELL_NEG: C102.2, J4.2 (Pin_2), Q2.1 (Pin_1), Q2.2 (Pin_2), Q2.3 (Pin_3), R106.2, TP102.1, U14.4 (VSS)
- new net CELL_POS: C104.1, C120.1, C121.1, J4.1 (Pin_1), R104.1, TP101.1, U5.2 (BAT), U5.3 (BAT), U8.3 (Pin_3)
- new net CHARGER_CHG_N: R110.1, U5.9 (~{CHG}), U9.5 (P01)
- new net CHARGER_PGOOD_N: R109.1, U5.7 (~{PGOOD}), U9.6 (P02)
- new net CHG_DISABLE: R126.1, U18.5 (P1), U5.4 (~{CE})
- new net CHG_ILIM: R111.1, U5.12 (ILIM)
- new net CHG_ISET: R113.1, U5.16 (ISET)
- new net CHG_ITERM: R112.1, U5.15 (ITERM)
- new net CHG_TMR: R114.1, U5.14 (TMR)
- new net CHG_TS: R108.1, U5.1 (TS)
- new net ESP_EN: C201.1, R203.1, SW1.1, U1.3 (EN)
- new net EX0: J5.15 (Pin_15), U9.13 (P10)
- new net EX1: J5.16 (Pin_16), U9.14 (P11)
- new net EX2: J5.17 (Pin_17), U9.15 (P12)
- new net EX3: J5.18 (Pin_18), U9.16 (P13)
- new net EX4: J5.19 (Pin_19), U9.17 (P14)
- new net EX5: J5.20 (Pin_20), U9.18 (P15)
- new net EX6: J5.21 (Pin_21), U9.19 (P16)
- new net EX7: J5.22 (Pin_22), U9.20 (P17)
- new net FG_ALERT_N: R125.1, U8.5 (Pin_5), U9.8 (P04)
- new net GND: C101.2, C103.2, C104.2, C105.2, C106.2, C107.2, C108.2, C109.2, C110.2, C111.2, C112.2, C114.2, C115.2, C116.2, C117.2, C118.2, C119.2, C120.2, C121.2, C122.2, C123.2, C124.2, C201.2, C202.2, C203.2, C301.2, C302.2, C303.2, C304.2, C305.2, C306.2, C307.2, C308.2, C309.2, C311.2, C312.2, C401.2, C402.2, C501.2, C502.2, C503.2, C504.2, C510.2, C511.2, C601.2, C602.2, C603.2, C604.2, C605.2, C606.2, C701.2, C702.2, C703.2, C704.2, C705.2, C706.2, C707.2, D101.1 (A1), D501.1 (A1), J1.A1 (GND), J1.A12 (GND), J1.B1 (GND), J1.B12 (GND), J2.6 (VSS), J2.9 (DET_B), J2.SH (SHIELD), J3.2 (Ext), J5.2 (Pin_2), J5.28 (Pin_28), J5.30 (Pin_30), J6.2 (Ext), LED1.3 (VSS), LED2.3 (VSS), LED3.3 (VSS), LED4.3 (VSS), Q1.2 (S), Q3.1 (Pin_1), Q3.2 (Pin_2), Q3.3 (Pin_3), Q4.2 (S), R101.2, R102.2, R103.2, R105.2, R107.2, R108.2, R111.2, R112.2, R113.2, R114.2, R115.2, R118.2, R121.2, R122.2, R123.2, R126.2, R127.2, R128.2, R603.2, R607.2, SW1.2, SW2.2, SW3.2, SW4.2, TP104.1, U1.1 (GND), U1.40 (GND), U1.41 (GND), U10.1 (Pin_1), U10.6 (Pin_6), U10.7 (Pin_7), U11.3 (Pin_3), U11.5 (Pin_5), U11.8 (Pin_8), U11.9 (Pin_9), U12.4 (VSS), U13.1 (Pin_1), U13.4 (Pin_4), U15.2 (Pin_2), U16.2 (GND), U17.2 (Pin_2), U18.2 (A1), U18.3 (A2), U18.8 (GND), U2.1 (DVSS), U2.11 (AVSS), U2.17 (I1), U2.18 (TESTEN), U2.3 (TVSS1), U2.41 (AVSS), U2.7 (TVSS2), U3.1 (Pin_1), U3.11 (Pin_11), U3.12 (Pin_12), U3.2 (Pin_2), U3.20 (Pin_20), U3.22 (Pin_22), U3.3 (Pin_3), U3.4 (Pin_4), U3.5 (Pin_5), U4.1 (GND), U4.10 (GND), U4.12 (GND), U5.17 (VSS), U5.8 (VSS), U6.10 (Pin_10), U6.15 (Pin_15), U6.4 (Pin_4), U7.4 (Pin_4), U8.1 (Pin_1), U8.4 (Pin_4), U8.6 (Pin_6), U8.9 (Pin_9), U9.12 (GND), U9.2 (A1), U9.21 (A0), U9.3 (A2), Y301.2 (Pin_2), Y301.4 (Pin_4)
- new net GNSS_3V3: C501.1, C502.1, R501.2, R502.2, R503.1, U17.6 (Pin_6), U4.7 (VCC_IO), U4.8 (VCC)
- new net GNSS_ANT_FEED: D501.2 (A2), J3.1 (In), L501.2, R504.2, TP501.1
- new net GNSS_BACKUP: C503.1, R503.2, U4.6 (V_BCKP)
- new net GNSS_BIAS: C504.1, L501.1, R505.2
- new net GNSS_LNA_EN: TP502.1, U4.13 (LNA_EN)
- new net GNSS_POWER_EN: U17.3 (Pin_3), U18.9 (P4)
- new net GNSS_QOD: R501.1, U17.5 (Pin_5)
- new net GNSS_RESET_N: R502.1, U4.9 (~{RESET})
- new net GNSS_RF: R504.1, U4.11 (RF_IN)
- new net GNSS_RX_FROM_MODULE: U1.23 (IO21), U4.2 (TXD)
- new net GNSS_TIMEPULSE: U1.11 (IO18), U4.4 (TIMEPULSE)
- new net GNSS_TX_TO_MODULE: U1.28 (IO35), U4.3 (RXD)
- new net GNSS_VCC_RF: R505.1, U4.14 (VCC_RF)
- new net GPIO1: J5.3 (Pin_3), R710.2
- new net GPIO1_MCU: R710.1, U1.39 (IO1)
- new net GPIO2: J5.4 (Pin_4), R711.2
- new net GPIO2_MCU: R711.1, U1.38 (IO2)
- new net GPIO4: J5.5 (Pin_5), R712.2
- new net GPIO40: J5.8 (Pin_8), R715.2
- new net GPIO40_MCU: R715.1, U1.33 (IO40)
- new net GPIO41: J5.9 (Pin_9), R716.2
- new net GPIO41_MCU: R716.1, U1.34 (IO41)
- new net GPIO42: J5.10 (Pin_10), R717.2
- new net GPIO42_MCU: R717.1, U1.35 (IO42)
- new net GPIO43: J5.11 (Pin_11), R718.2
- new net GPIO43_MCU: R718.1, U1.37 (TXD0)
- new net GPIO44: J5.12 (Pin_12), R719.2
- new net GPIO44_MCU: R719.1, U1.36 (RXD0)
- new net GPIO47: J5.13 (Pin_13), R720.2
- new net GPIO47_MCU: R720.1, U1.24 (IO47)
- new net GPIO48: J5.14 (Pin_14), R721.2
- new net GPIO48_MCU: R721.1, U1.25 (IO48)
- new net GPIO4_MCU: R712.1, U1.4 (IO4)
- new net GPIO8: J5.6 (Pin_6), R713.2
- new net GPIO8_MCU: R713.1, U1.12 (IO8)
- new net GPIO9: J5.7 (Pin_7), R714.2
- new net GPIO9_MCU: R714.1, U1.17 (IO9)
- new net I2C_SCL: J5.24 (Pin_24), R702.1, U1.6 (IO6), U10.13 (Pin_13), U11.2 (Pin_2), U12.6 (SCL), U18.14 (SCL), U2.27 (NSS/P50_SCL/HSU_RX), U8.7 (Pin_7), U9.22 (SCL)
- new net I2C_SDA: J5.23 (Pin_23), R701.1, U1.5 (IO5), U10.14 (Pin_14), U11.4 (Pin_4), U12.5 (SDA), U18.15 (SDA), U2.28 (MOSI/SDA/HSU_TX), U8.8 (Pin_8), U9.23 (SDA)
- new net IOEXP_INT_N: R703.1, U1.32 (IO39), U18.13 (~{INT}), U9.1 (~{INT})
- new net IR_GATE: Q1.1 (G), R602.2, R603.1
- new net IR_LED_A: D1.2 (A), R601.2
- new net IR_LED_K: D1.1 (K), Q1.3 (D)
- new net IR_RX: U1.30 (IO37), U13.3 (Pin_3)
- new net IR_RX_VS: C601.1, C602.1, R604.2, U13.2 (Pin_2)
- new net IR_TX: R602.1, U1.29 (IO36)
- new net JTAG_STRAP_TP: TP201.1, U1.15 (IO3)
- new net NFC_AVDD: C302.1, FB301.2, U2.8 (AVDD)
- new net NFC_DVDD: C304.1, R301.2, U2.39 (DVDD)
- new net NFC_I0: R301.1, U2.16 (I0)
- new net NFC_IRQ_N: U1.7 (IO7), U2.25 (P70_IRQ)
- new net NFC_LOADMOD: TP301.1, U2.2 (LOADMOD)
- new net NFC_LOOP_A: AE1.1, C310.1, C311.1, R303.2, R305.1
- new net NFC_LOOP_B: AE1.2, C310.2, C312.1, R304.2
- new net NFC_OSCIN: C306.1, U2.14 (OSCIN), Y301.1 (Pin_1)
- new net NFC_OSCOUT: C307.1, U2.15 (OSCOUT), Y301.3 (Pin_3)
- new net NFC_RESET_N: R302.1, U18.7 (P3), U2.38 (~{RSTPD})
- new net NFC_RX: R305.2, U2.10 (RX)
- new net NFC_SVDD: C305.1, U2.37 (SVDD)
- new net NFC_TX1: L301.1, U2.4 (TX1)
- new net NFC_TX1_F: C308.1, L301.2, R303.1
- new net NFC_TX2: L302.1, U2.6 (TX2)
- new net NFC_TX2_F: C309.1, L302.2, R304.1
- new net NFC_VMID: C301.1, U2.9 (VMID)
- new net PWR_3V3_PG: R119.1, U6.2 (Pin_2)
- new net RGB_D1_2: LED1.2 (DOUT), LED2.4 (DIN)
- new net RGB_D2_3: LED2.2 (DOUT), LED3.4 (DIN)
- new net RGB_D3_4: LED3.2 (DOUT), LED4.4 (DIN)
- new net RGB_DATA: R605.1, U1.18 (IO10)
- new net RGB_DIN1: LED1.4 (DIN), R605.2
- new net RGB_DOUT4: LED4.2 (DOUT), TP601.1
- new net RTC_OSCI: U12.1 (OSCI), Y701.1
- new net RTC_OSCO: U12.2 (OSCO), Y701.2
- new net SD_CS_DEV: J2.2 (DAT3/CD), R510.2, R515.1
- new net SD_CS_N: R510.1, U1.10 (IO17)
- new net SD_DAT1: J2.8 (DAT1), R518.1
- new net SD_DAT2: J2.1 (DAT2), R514.1
- new net SD_DETECT_N: J2.10 (DET_A), R519.1, U9.4 (P00)
- new net SD_MISO: J2.7 (DAT0), R513.2, R517.1
- new net SD_MOSI: J2.3 (CMD), R511.2, R516.1
- new net SD_SCK: J2.5 (CLK), R512.2
- new net SPI_MISO: J5.27 (Pin_27), R403.1, R513.1, U1.21 (IO13)
- new net SPI_MOSI: J5.26 (Pin_26), R402.1, R511.1, U1.19 (IO11)
- new net SPI_SCK: J5.25 (Pin_25), R401.1, R512.1, U1.20 (IO12)
- new net STRAP_BOOT_TP: TP202.1, U1.16 (IO46)
- new net STRAP_VDD_SPI_TP: TP203.1, U1.26 (IO45)
- new net SUBGHZ_ANT: J6.1 (In), R405.2
- new net SUBGHZ_CS_N: R404.1, U1.22 (IO14)
- new net SUBGHZ_GDO0: U1.8 (IO15), U3.15 (Pin_15)
- new net SUBGHZ_GDO2: U1.9 (IO16), U3.14 (Pin_14)
- new net SUBGHZ_RF: R405.1, U3.21 (Pin_21)
- new net SUB_CS_N: R404.2, U3.19 (Pin_19)
- new net SUB_MISO: R403.2, U3.16 (Pin_16)
- new net SUB_MOSI: R402.2, U3.17 (Pin_17)
- new net SUB_SCK: R401.2, U3.18 (Pin_18)
- new net U15_ILIM: R123.1, U15.5 (Pin_5)
- new net U6_FB: R117.2, R118.1, U6.5 (Pin_5)
- new net U6_L1: L6.1, U6.11 (Pin_11)
- new net U6_L2: L6.2, U6.9 (Pin_9)
- new net U6_PS_SYNC: R116.2, U6.1 (Pin_1)
- new net U6_VAUX: C107.1, U6.3 (Pin_3)
- new net U7_FB: C113.2, R120.2, R121.1, U7.1 (Pin_1)
- new net U7_SW: L7.2, U7.5 (Pin_5)
- new net USB_CC1: J1.A5 (CC1), R101.1, U16.4 (I/O3)
- new net USB_CC2: J1.B5 (CC2), R102.1, U16.6 (I/O4)
- new net USB_DM_CONN: J1.A7 (D-), J1.B7 (D-), R201.1, U16.3 (I/O2)
- new net USB_DP_CONN: J1.A6 (D+), J1.B6 (D+), R202.1, U16.1 (I/O1)
- new net USB_D_N: R201.2, U1.13 (USB_D-)
- new net USB_D_P: R202.2, U1.14 (USB_D+)
- new net USB_SHIELD: C101.1, J1.SH (SHIELD), R103.1
- new net USER_BUTTON_A_N: R608.1, SW3.1, U18.11 (P6)
- new net USER_BUTTON_B_N: R609.1, SW4.1, U18.12 (P7)
- new net VBUS_FUSED: C103.1, C106.1, D101.2 (A2), F1.2, U16.5 (VBUS), U5.13 (IN)
- new net VBUS_USB: F1.1, J1.A4 (VBUS), J1.A9 (VBUS), J1.B4 (VBUS), J1.B9 (VBUS)
- new net VSYS: C105.1, C108.1, C109.1, C114.1, C122.1, C123.1, L7.1, R116.1, U5.10 (OUT), U5.11 (OUT), U6.12 (Pin_12), U6.13 (Pin_13), U6.14 (Pin_14), U7.3 (Pin_3)
- no-connect marks 0 -> 36
Other:
- removed sheet 01_USB_POWER
- removed sheet 02_MCU
- removed sheet 03_NFC
- removed sheet 04_SUBGHZ
- removed sheet 05_GNSS_SD
- removed sheet 06_IR_UI
- removed sheet 07_SENSORS_IO
- note added: "01 USB / BATTERY / POWER"
- note added: "02 ESP32-S3 MCU / USB"
- note added: "03 PN532 NFC / TUNABLE LOOP"
- note added: "04 E07 CC1101 SUB-GHZ"
- note added: "05 GNSS / ANTENNA / MICROSD"
- note added: "06 IR / RGB / BUTTONS / BUZZER"
- note added: "07 SENSORS / RTC / IO EXPANSION"
- company: (none) -> PocketLab
- title: PocketLab Card V1 -> PocketLab Card V1 - Complete Electrical Capture

Commit message: Save full hardware placement checkpoint
Parts:
- removed C503: 100uF low-leak, Capacitor_SMD:C_1210_3225Metric, symbol Device:C
- removed D101: SMF5.0A, Diode_SMD:D_SOD-123F, symbol Device:D_TVS
- removed FB301: 600R@100MHz, Inductor_SMD:L_0805_2012Metric, symbol Device:FerriteBead
- removed J6: SUB-GHz ANT U.FL, Connector_Coaxial:U.FL_Hirose_U.FL-R-SMT-1_Vertical, symbol Connector:Conn_Coaxial
- removed R405: 0R ANT SELECT, Resistor_SMD:R_0805_2012Metric, symbol Device:R
- removed R503: 100R, Resistor_SMD:R_0805_2012Metric, symbol Device:R
- removed R504: 0R RF, Resistor_SMD:R_0805_2012Metric, symbol Device:R
- removed TP501: GNSS RF TEST, TestPoint:TestPoint_Pad_D1.0mm, symbol Connector:TestPoint
- added C313: 10uF DVDD bulk, Capacitor_SMD:C_0805_2012Metric, symbol Device:C
- added C314: 100nF TVDD, Capacitor_SMD:C_0805_2012Metric, symbol Device:C
- added C315: 4.7uF TVDD bulk, Capacitor_SMD:C_0805_2012Metric, symbol Device:C
- added C316: 100nF PVDD, Capacitor_SMD:C_0805_2012Metric, symbol Device:C
- added C317: 100nF VBAT, Capacitor_SMD:C_0805_2012Metric, symbol Device:C
- added C318: 1nF C0G RX COUPLING, Capacitor_SMD:C_0603_1608Metric, symbol Device:C
- added C512: 47uF 6.3V LOW-ESR, Capacitor_SMD:C_1210_3225Metric, symbol Device:C
- added D101: SMF5.0A, Diode_SMD:D_SOD-123F, symbol Device:D_Zener
- added J7: OPTIONAL 10k NTC - CUT SJ1, Connector_PinHeader_2.54mm:PinHeader_1x02_P2.54mm_Vertical, symbol Connector_Generic:Conn_01x02
- added R306: 1k VMID BIAS, Resistor_SMD:R_0805_2012Metric, symbol Device:R
- added R406: 100k CS SAFE-HIGH, Resistor_SMD:R_0805_2012Metric, symbol Device:R
- added R506: 100k SAFE-OFF, Resistor_SMD:R_0805_2012Metric, symbol Device:R
- added R507, R508: 1k UART BACKPOWER LIMIT, Resistor_SMD:R_0805_2012Metric, symbol Device:R
- added R722, R723, R724, R725, R726, R727, R728, R729: 220R EXPANSION PROTECTION, Resistor_SMD:R_0805_2012Metric, symbol Device:R
- added R730, R731, R732, R733, R734: 100R, Resistor_SMD:R_0805_2012Metric, symbol Device:R
- added SJ1: TS FIXED / CUT FOR EXT NTC, Jumper:SolderJumper-2_P1.3mm_Bridged_RoundedPad1.0x1.5mm, symbol Jumper:SolderJumper_2_Bridged
- added TP105: POWER VBUS_USB, TestPoint:TestPoint_Pad_D1.0mm, symbol Connector:TestPoint
- added TP106: POWER VBUS_FUSED, TestPoint:TestPoint_Pad_D1.0mm, symbol Connector:TestPoint
- added TP107: POWER VSYS, TestPoint:TestPoint_Pad_D1.0mm, symbol Connector:TestPoint
- added TP108: POWER +3V3, TestPoint:TestPoint_Pad_D1.0mm, symbol Connector:TestPoint
- added TP109: POWER +5V_RAW, TestPoint:TestPoint_Pad_D1.0mm, symbol Connector:TestPoint
- added TP110: POWER +5V_AUX, TestPoint:TestPoint_Pad_D1.0mm, symbol Connector:TestPoint
- added U19: SRV05-4MR6T1G SD ESD, Package_TO_SOT_SMD:SOT-23-6, symbol Power_Protection:SRV05-4
- AE1: footprint (none) -> PocketLab_Custom:NFC_Loop_35x27mm_4T_TUNE
- C109, C310, C311, C312: DNP (none) -> true
- C302: value 100nF -> 100nF AVDD
- C303: value 4.7uF -> 4.7uF VBAT bulk
- C504: value 10nF -> 10nF DNP ACTIVE-ANT BIAS; DNP (none) -> true
- D501: value Low-cap RF ESD -> TPD1E0B04 0.13pF RF ESD; footprint Diode_SMD:D_SOD-523 -> Package_SON:Texas_DPY0002A_0.6x1mm_P0.65mm; MPN (none) -> TPD1E0B04DPYR; Manufacturer (none) -> TI
- L501: value 27nH high-Q -> 27nH high-Q DNP ACTIVE-ANT BIAS; DNP (none) -> true
- R302: value 10k -> 10k RESET default asserted
- R305: value 1k RX TAP -> 2.7k RX TAP
- R505: value 10R 0.25W -> 10R 0.25W DNP ACTIVE-ANT BIAS; DNP (none) -> true
- R701, R702: value 4.7k -> 3.3k
- U3: value E07-900M10S 868MHz -> E07-900M10S IPEX 868MHz
- Y701: value 32.768kHz 12.5pF -> 32.768kHz CL=7pF; MPN (none) -> ABS07-32.768KHZ-7-T; Manufacturer (none) -> Abracon
Connections:
- net GNSS_RF is gone; now on net GNSS_ANT_FEED: U4.11 (RF_IN)
- net NFC_AVDD is gone; now on net NFC_DVDD: C302.1, U2.8 (AVDD)
- net +3V3: now also C316.1, C317.1, C512.1, R406.2, TP108.1, U19.5 (VP); no longer R302.2, U2.5 (TVDD)
- net +5V_AUX: now also TP110.1
- net +5V_RAW: now also TP109.1
- net CHG_TS: now also J7.1 (Pin_1), SJ1.1 (A); no longer R108.1
- net EX0: now also R722.2; no longer U9.13 (P10)
- net EX1: now also R723.2; no longer U9.14 (P11)
- net EX2: now also R724.2; no longer U9.15 (P12)
- net EX3: now also R725.2; no longer U9.16 (P13)
- net EX4: now also R726.2; no longer U9.17 (P14)
- net EX5: now also R727.2; no longer U9.18 (P15)
- net EX6: now also R728.2; no longer U9.19 (P16)
- net EX7: now also R729.2; no longer U9.20 (P17)
- net GND: now also R302.2, C313.2, C314.2, C315.2, C316.2, C317.2, C512.2, D101.2 (A), J7.2 (Pin_2), R506.2, U19.2 (VN)
- net GNSS_POWER_EN: now also R506.1
- net GNSS_RX_FROM_MODULE: now also R507.1; no longer U4.2 (TXD)
- net GNSS_TX_TO_MODULE: now also R508.1; no longer U4.3 (RXD)
- net I2C_SCL: now also R731.1; no longer J5.24 (Pin_24)
- net I2C_SDA: now also R730.1; no longer J5.23 (Pin_23)
- net NFC_DVDD: now also U2.5 (TVDD), C313.1, C314.1, C315.1
- net NFC_RX: now also C318.2, R306.2; no longer R305.2
- net NFC_VMID: now also R306.1
- net SD_CS_DEV: now also U19.1 (IO1)
- net SD_MISO: now also U19.6 (IO4)
- net SD_MOSI: now also U19.3 (IO2)
- net SD_SCK: now also U19.4 (IO3)
- net SPI_MISO: now also R734.1; no longer J5.27 (Pin_27)
- net SPI_MOSI: now also R733.1; no longer J5.26 (Pin_26)
- net SPI_SCK: now also R732.1; no longer J5.25 (Pin_25)
- net SUB_CS_N: now also R406.1
- net VBUS_FUSED: now also D101.1 (K), TP106.1
- net VBUS_USB: now also TP105.1
- net VSYS: now also TP107.1
- net GNSS_BACKUP: no longer names the net of U4.6 (V_BCKP)
- net SUBGHZ_RF: no longer names the net of U3.21 (Pin_21)
- net USB_DM_CONN renamed USB_CONN_N
- net USB_DP_CONN renamed USB_CONN_P
- new net CHG_TS_FIXED: R108.1, SJ1.2 (B)
- new net EX0_INT: R722.1, U9.13 (P10)
- new net EX1_INT: R723.1, U9.14 (P11)
- new net EX2_INT: R724.1, U9.15 (P12)
- new net EX3_INT: R725.1, U9.16 (P13)
- new net EX4_INT: R726.1, U9.17 (P14)
- new net EX5_INT: R727.1, U9.18 (P15)
- new net EX6_INT: R728.1, U9.19 (P16)
- new net EX7_INT: R729.1, U9.20 (P17)
- new net GNSS_UART_RX_MOD: R508.2, U4.3 (RXD)
- new net GNSS_UART_TX_MOD: R507.2, U4.2 (TXD)
- new net I2C_SCL_HDR: J5.24 (Pin_24), R731.2
- new net I2C_SDA_HDR: J5.23 (Pin_23), R730.2
- new net NFC_RX_AC: C318.1, R305.2
- new net SPI_MISO_HDR: J5.27 (Pin_27), R734.2
- new net SPI_MOSI_HDR: J5.26 (Pin_26), R733.2
- new net SPI_SCK_HDR: J5.25 (Pin_25), R732.2
- no-connect marks 36 -> 38

Commit message: Save integrated card hardware and firmware checkpoint
Parts:
- removed BZ1: PKMCS0909E, Buzzer_Beeper:Buzzer_Murata_PKMCS0909E, symbol Device:Buzzer
- removed J7: OPTIONAL 10k NTC - CUT SJ1, Connector_PinHeader_2.54mm:PinHeader_1x02_P2.54mm_Vertical, symbol Connector_Generic:Conn_01x02
- removed Q4: AO3400A BUZZER, Package_TO_SOT_SMD:SOT-23, symbol Transistor_FET:AO3400A
- removed R607: 100k, Resistor_SMD:R_0805_2012Metric, symbol Device:R
- removed U3: E07-900M10S IPEX 868MHz, PocketLab_Custom:E07-900M10S, symbol Connector_Generic:Conn_02x11_Odd_Even
- added A1: T3-868M SPRING ANTENNA, PocketLab_Custom:T3-868M_Edge_Solder, symbol Device:Antenna
- added C403, C404: DNP SUBGHZ MATCH, Capacitor_SMD:C_0805_2012Metric, symbol Device:C
- added C607, C617: 22uF 10V X5R IR BUFFER, Capacitor_SMD:C_1206_3216Metric, symbol Device:C
- added C608: 100nF IR HF, Capacitor_SMD:C_0805_2012Metric, symbol Device:C
- added C609, C612, C616: 100nF X7R, Capacitor_SMD:C_0805_2012Metric, symbol Device:C
- added C610, C611: 1uF X7R, Capacitor_SMD:C_0805_2012Metric, symbol Device:C
- added C613, C615: 4.7uF X5R, Capacitor_SMD:C_0805_2012Metric, symbol Device:C
- added C614: 2.2uF X7R, Capacitor_SMD:C_0805_2012Metric, symbol Device:C
- added D2, D3: TSAL6200 940nm, PocketLab_Custom:TSAL6200_LayFlat_Inboard, symbol Device:LED
- added J8: ER-OLED0.42-1W 72x40 SSD1306B, PocketLab_Custom:EastRising_ER-OLED0.42-1W_SolderFPC, symbol Connector_Generic:Conn_01x16
- added J9: GPIO38 2.54mm DUPONT, Connector_PinHeader_2.54mm:PinHeader_1x01_P2.54mm_Vertical, symbol Connector_Generic:Conn_01x01
- added R405: 0R SUBGHZ MATCH, Resistor_SMD:R_0805_2012Metric, symbol Device:R
- added R610, R611: 39R 0.5W pulse-rated, Resistor_SMD:R_1210_3225Metric, symbol Device:R
- added R735: 100k EN pull-down, Resistor_SMD:R_0805_2012Metric, symbol Device:R
- added SW5: MAIN POWER OFF / ON, Button_Switch_SMD:SW_SPDT_Shouhan_MSK12C02, symbol Switch:SW_SPDT
- added U20: SN74AHCT1G126DBVR RGB LEVEL SHIFT, Package_TO_SOT_SMD:SOT-23-5, symbol 74xGxx:74AHCT1G126
- added U3: E07-900MM10S 855-925MHz, PocketLab_Custom:E07-900MM10S, symbol Connector_Generic:Conn_02x10_Odd_Even
- AE1, SJ1, TP101, TP102, TP103, TP104, TP105, TP106, TP107, TP108, TP109, TP110, TP201, TP202, TP203, TP301, TP502, TP601, TP701, TP702, TP703: now left out of the parts list
- C109, C310, C311, C312, C504, L501, R505: now not fitted
- D1: footprint LED_THT:LED_D5.0mm -> PocketLab_Custom:TSAL6200_LayFlat_Inboard; Assembly (none) -> MANUAL_EDGE_BEND; LCSC (none) -> C55528
- J5: value 2x15 2.54mm DUPONT EXPANSION -> 30-PIN 2.54mm DUPONT GRID; footprint Connector_PinHeader_2.54mm:PinHeader_2x15_P2.54mm_Vertical -> PocketLab_Custom:Dupont_Grid_6x5_P2.54mm
- LED1, LED2, LED3, LED4: value WS2812B-MINI-V3 -> WS2812B-2020; footprint LED_SMD:LED_WS2812B-Mini_PLCC4_3.5x3.5mm -> LED_SMD:LED_WS2812B-2020_PLCC4_2.0x2.0mm; LCSC (none) -> C965555; MPN (none) -> WS2812B-2020; Manufacturer (none) -> Worldsemi
- Q2, Q3: footprint Package_SON:VSON-8_3.3x3.3mm_P0.65mm_NexFET -> PocketLab_Custom:CSD16406Q3_VSON-8_3.3x3.3mm_P0.65mm_JLC
- R601: value 39R 1W pulse-rated -> 39R 0.5W pulse-rated; footprint Resistor_SMD:R_2512_6332Metric -> Resistor_SMD:R_1210_3225Metric
- R605: value 330R -> 68R
- R606: value 100R -> 100R GPIO38 PROTECTION
- SW1, SW2: footprint Button_Switch_SMD:SW_SPST_TL3305A -> Button_Switch_SMD:SW_Push_1P1T_NO_CK_KMR2; LCSC (none) -> C72443; MPN (none) -> KMR221GLFS; Manufacturer (none) -> C&K
- U1: footprint RF_Module:ESP32-S3-WROOM-1 -> PocketLab_Card:ESP32-S3-WROOM-1_PhysicalCourtyard
Connections:
- net +3V3: now also C612.1, C613.1, J8.5 (Pin_5), J8.7 (Pin_7), J8.8 (Pin_8), U3.1 (Pin_1); no longer C603.1, C604.1, C605.1, C606.1, LED1.1 (VDD), LED2.1 (VDD), LED3.1 (VDD), LED4.1 (VDD)
- net +5V_RAW: now also C603.1, C604.1, C605.1, C606.1, LED1.1 (VDD), LED2.1 (VDD), LED3.1 (VDD), LED4.1 (VDD), C607.1, C608.1, C609.1, C617.1, R610.1, R611.1, U20.5 (VCC)
- net BOOST5_EN: now also U20.1
- net CHG_TS: now also J5.28 (Pin_28)
- net ESP_EN: now also J8.10 (Pin_10)
- net GND: now also C403.2, C404.2, C607.2, C608.2, C609.2, C612.2, C613.2, C614.2, C615.2, C616.2, C617.2, J8.11 (Pin_11), J8.6 (Pin_6), J8.9 (Pin_9), R735.2, SW5.1 (A), U20.3 (GND), U3.16 (Pin_16), U3.2 (Pin_2), U3.7 (Pin_7); no longer J5.28 (Pin_28)
- net I2C_SCL: now also J8.12 (Pin_12)
- net I2C_SDA: now also J8.13 (Pin_13), J8.14 (Pin_14)
- net IR_LED_K: now also D2.1 (K), D3.1 (K)
- net RGB_DATA: now also U20.2; no longer R605.1
- net SUBGHZ_GDO0: now also U3.18 (Pin_18)
- net SUBGHZ_GDO2: now also U3.20 (Pin_20)
- net SUB_CS_N: now also U3.14 (Pin_14)
- net SUB_MISO: now also U3.12 (Pin_12)
- net SUB_MOSI: now also U3.13 (Pin_13)
- net SUB_SCK: now also U3.15 (Pin_15)
- net U6_PS_SYNC: now also U6.14 (Pin_14), R735.1, SW5.2 (B); no longer R116.2
- net VSYS: no longer U6.14 (Pin_14)
- net BUZZER_GATE renamed GPIO38
- net GPIO38: now also J9.1 (Pin_1)
- net BUZZER_PWM renamed GPIO38_MCU
- net IR_LED_A renamed IR_LED_A1
- new net IR_LED_A2: D2.2 (A), R610.2
- new net IR_LED_A3: D3.2 (A), R611.2
- new net OLED_C1N: C611.2, J8.4 (Pin_4)
- new net OLED_C1P: C611.1, J8.3 (Pin_3)
- new net OLED_C2N: C610.2, J8.2 (Pin_2)
- new net OLED_C2P: C610.1, J8.1 (Pin_1)
- new net OLED_VCC: C615.1, C616.1, J8.16 (Pin_16)
- new net OLED_VCOMH: C614.1, J8.15 (Pin_15)
- new net PWR_SW_ON: R116.2, SW5.3 (C)
- new net RGB_BUF_5V: R605.1, U20.4
- new net SUBGHZ_RF_ANT: A1.1 (A), C404.1, R405.2
- new net SUBGHZ_RF_MOD: C403.1, R405.1, U3.6 (Pin_6)
- no-connect marks 38 -> 41
Other:
- note added: "06 IR / RGB / BUTTONS / OLED"
- note removed: "06 IR / RGB / BUTTONS / BUZZER"
