File: hardware/PocketLab-Card.kicad_sch (KiCad schematic)
At the start: 252 parts, among them J1 USB-C DATA/POWER, J2 microSD, J3 GNSS ANT U.FL, J4 PROTECTED 1S LiPo 3.7V, J5 30-PIN 2.54mm DUPONT GRID, J8 ER-OLED0.42-1W 72x40 SSD1306B, J9 GPIO38 2.54mm DUPONT, Q1 AO3400A IR DRIVER, Q2 CSD16406Q3 DISCHARGE, Q3 CSD16406Q3 CHARGE, SW1 RESET, SW2 BOOT, SW3 USER A, SW4 USER B, SW5 MAIN POWER OFF / ON, U1 ESP32-S3-WROOM-1-N8R2, U10 BMI270 (FULL OPTION), U11 BMP390 (FULL OPTION), U12 PCF8563T, U13 TSOP75338WTR 38kHz, U14 BQ29700DSE, U15 TPS2553DBVR 500mA LIMIT, U16 USBLC6-4SC6Y, U17 TPS22919DCKR GNSS LOAD SWITCH, U18 TCA9534PWR INTERNAL CONTROL, U19 SRV05-4MR6T1G SD ESD, U2 PN5321A3HN/C106, U20 SN74AHCT1G126DBVR RGB LEVEL S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, U3 E07-900MM10S 855-925MHz, U4 MAX-M10S-00B, U5 BQ24074RGTR, U6 TPS63070RNMR 3V3, U7 TPS61023DRLR 5V BOOST, U8 MAX17048G+T10, U9 TCA9535PWR, Y301 27.12MHz crystal (pins 2/4 sh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, Y701 32.768kHz CL=7pF

Commit message: Save RFID and critical routing checkpoint
Parts:
- removed D501: TPD1E0B04 0.13pF RF ESD, Package_SON:Texas_DPY0002A_0.6x1mm_P0.65mm, symbol Device:D_TVS
- removed J3: GNSS ANT U.FL, Connector_Coaxial:U.FL_Hirose_U.FL-R-SMT-1_Vertical, symbol Connector:Conn_Coaxial
- removed J9: GPIO38 2.54mm DUPONT, Connector_PinHeader_2.54mm:PinHeader_1x01_P2.54mm_Vertical, symbol Connector_Generic:Conn_01x01
- removed L501: 27nH high-Q DNP ACTIVE-ANT BIAS, Inductor_SMD:L_0805_2012Metric, symbol Device:L
- removed R505: 10R 0.25W DNP ACTIVE-ANT BIAS, Resistor_SMD:R_0805_2012Metric, symbol Device:R
- removed R507, R508: 1k UART BACKPOWER LIMIT, Resistor_SMD:R_0805_2012Metric, symbol Device:R
- removed TP601: RGB DOUT, TestPoint:TestPoint_Pad_D1.0mm, symbol Connector:TestPoint
- removed TP701: BMI INT1, TestPoint:TestPoint_Pad_D1.0mm, symbol Connector:TestPoint
- removed TP702: BMP INT, TestPoint:TestPoint_Pad_D1.0mm, symbol Connector:TestPoint
- removed TP703: BMI INT2, TestPoint:TestPoint_Pad_D1.0mm, symbol Connector:TestPoint
- removed U4: MAX-M10S-00B, RF_GPS:ublox_MAX, symbol RF_GPS:MAX-M10S
- added C503: 100nF CEXT, Capacitor_SMD:C_0805_2012Metric, symbol Device:C
- added C505: 100nF C0G COIL ISOLATION, Capacitor_SMD:C_0805_2012Metric, symbol Device:C
- added C506: 3.9nF C0G LF RESONANCE, Capacitor_SMD:C_0805_2012Metric, symbol Device:C
- added C507: 100pF C0G DNP LF TUNE, Capacitor_SMD:C_0603_1608Metric, symbol Device:C
- added C508: 220pF C0G DNP LF TUNE, Capacitor_SMD:C_0603_1608Metric, symbol Device:C
- added C509: 10pF C0G DNP RX EMI, Capacitor_SMD:C_0603_1608Metric, symbol Device:C
- added C513: 100nF OSC supply, Capacitor_SMD:C_0805_2012Metric, symbol Device:C
- added C515: 100nF AHCT supply, Capacitor_SMD:C_0805_2012Metric, symbol Device:C
- added C516: 100nF LVC supply, Capacitor_SMD:C_0805_2012Metric, symbol Device:C
- added C517: 100nF secure element, Capacitor_SMD:C_0805_2012Metric, symbol Device:C
- added J3: EXTERNAL 400uH LF COIL, Connector_PinHeader_2.54mm:PinHeader_1x02_P2.54mm_Vertical, symbol Connector_Generic:Conn_01x02
- added R503: 1k LF EMI RETURN, Resistor_SMD:R_0805_2012Metric, symbol Device:R
- added R504: 150k 1% RX DIVIDER, Resistor_SMD:R_0805_2012Metric, symbol Device:R
- added R509: 10k PAIR pull-up, Resistor_SMD:R_0805_2012Metric, symbol Device:R
- added R607: 10k, Resistor_SMD:R_0603_1608Metric, symbol Device:R
- added R736: 10k 1% BOARD TEMP BIAS, Resistor_SMD:R_0603_1608Metric, symbol Device:R
- added RT701: 10k NTC B3950 1%, Resistor_SMD:R_0603_1608Metric, symbol Device:Thermistor
- added SW6: PAIR, Button_Switch_SMD:SW_Push_1P1T_NO_CK_KMR2, symbol Switch:SW_Push
- added SW7: SELECT, Button_Switch_SMD:SW_Push_1P1T_NO_CK_KMR2, symbol Switch:SW_Push
- added U21: SN74AHCT125PWR LF 3V3-TO-5V, Package_SO:TSSOP-14_4.4x5mm_P0.65mm, symbol Connector_Generic:Conn_02x07_Odd_Even
- added U22: SN74LVC1G17DBVR LF 5V-TO-3V3, Package_TO_SOT_SMD:SOT-23-5_HandSoldering, symbol 74xGxx:74LVC1G17
- added U23: ATECC608C-SSHDA-T, Package_SO:SOIC-8_3.9x4.9mm_P1.27mm, symbol Security:ATECC608A-SSHDA
- added U24: SRV05-4MR6T1G J5 BUS ESD, Package_TO_SOT_SMD:SOT-23-6, symbol Power_Protection:SRV05-4
- added U25: SRV05-4MR6T1G J5 SPI ESD, Package_TO_SOT_SMD:SOT-23-6, symbol Power_Protection:SRV05-4
- added U4: HTRC11001T/03EE,11 125kHz, Package_SO:SO-14_3.9x8.65mm_P1.27mm, symbol RF_RFID:HTRC11001T
- added Y501: 4MHz 5V CMOS OSCILLATOR, Oscillator:Oscillator_SMD_EuroQuartz_XO32-4Pin_3.2x2.5mm_RotB_HandSoldering, symbol Connector_Generic:Conn_01x04
- C501: value 100nF -> 100nF HTRC supply
- C502: value 10uF -> 10uF HTRC pulse reservoir
- C504: value 10nF DNP ACTIVE-ANT BIAS -> 100nF QGND; footprint Capacitor_SMD:C_0603_1608Metric -> Capacitor_SMD:C_0805_2012Metric; DNP true -> (none); now fitted
- R502: value 10k -> 47R 0.5W ANTENNA CURRENT LIMIT; footprint Resistor_SMD:R_0805_2012Metric -> Resistor_SMD:R_1210_3225Metric
- R605, R608, R609, R710, R711, R712, R713, R715, R716, R717, R718, R719, R720, R721, R722, R723, R724, R725, R726, R727, R728, R729, R730, R731, R732, R733, R734: footprint Resistor_SMD:R_0805_2012Metric -> Resistor_SMD:R_0603_1608Metric
- R606: value 100R GPIO38 PROTECTION -> 100R PAIR GPIO PROTECTION; footprint Resistor_SMD:R_0805_2012Metric -> Resistor_SMD:R_0603_1608Metric
- R714: value 100R -> 100R BOARD TEMP PROBE; footprint Resistor_SMD:R_0805_2012Metric -> Resistor_SMD:R_0603_1608Metric
- SW3: value USER A -> UP; footprint Button_Switch_SMD:SW_SPST_TL3305A -> Button_Switch_SMD:SW_Push_1P1T_NO_CK_KMR2; LCSC (none) -> C72443; MPN (none) -> KMR221GLFS; Manufacturer (none) -> C&K
- SW4: value USER B -> DOWN; footprint Button_Switch_SMD:SW_SPST_TL3305A -> Button_Switch_SMD:SW_Push_1P1T_NO_CK_KMR2; LCSC (none) -> C72443; MPN (none) -> KMR221GLFS; Manufacturer (none) -> C&K
- TP502: value LNA ENABLE -> LF ANTENNA TAP - HIGH VOLTAGE
- U17: value TPS22919DCKR GNSS LOAD SWITCH -> TPS22919DCKR LF 5V LOAD SWITCH; LCSC (none) -> C2149796
Connections:
- net +3V3: now also C516.1, C517.1, R509.2, R607.2, R736.1, U22.5 (VCC), U23.8 (VCC), U24.5 (VP), U25.5 (VP); no longer U17.1 (Pin_1)
- net +5V_RAW: now also U17.1 (Pin_1)
- net GND: now also C503.2, C513.2, C515.2, C516.2, C517.2, R503.2, RT701.2, SW6.2, SW7.2, U21.1 (Pin_1), U21.12 (Pin_12), U21.4 (Pin_4), U21.7 (Pin_7), U21.9 (Pin_9), U22.3 (GND), U23.4 (GND), U24.2 (VN), U25.2 (VN), U4.1 (VSS), U4.5 (MODE), Y501.2 (Pin_2)
- net I2C_SCL: now also U23.6 (SCL)
- net I2C_SCL_HDR: now also U24.3 (IO2)
- net I2C_SDA: now also U23.5 (SDA)
- net I2C_SDA_HDR: now also U24.1 (IO1)
- net SPI_MISO_HDR: now also U25.1 (IO1)
- net SPI_MOSI_HDR: now also U25.3 (IO2)
- net SPI_SCK_HDR: now also U25.4 (IO3)
- net BMP_INT: no longer names the net of U11.7 (Pin_7)
- net BMP_INT: no longer U9.11 (P07)
- net GNSS_3V3 renamed LF_5V
- net LF_5V: now also C513.1, C515.1, U21.10 (Pin_10), U21.13 (Pin_13), U21.14 (Pin_14), U4.3 (VDD), Y501.1 (Pin_1), Y501.4 (Pin_4); no longer R502.2
- net GNSS_BIAS renamed LF_QGND
- net LF_QGND: now also C509.2, U4.13 (QGND)
- net GNSS_LNA_EN renamed LF_TAP
- net LF_TAP: now also R502.2, C506.1, C507.1, C508.1, R504.1
- net GNSS_POWER_EN renamed LF_RFID_EN
- net GNSS_QOD renamed LF_QOD
- net GNSS_RESET_N renamed LF_ANT_B
- net LF_ANT_B: now also J3.2 (Pin_2)
- net GNSS_RX_FROM_MODULE renamed LF_DOUT_3V3
- net LF_DOUT_3V3: now also U22.4
- net GNSS_TIMEPULSE renamed LF_SCLK_3V3
- net LF_SCLK_3V3: now also U21.2 (Pin_2)
- net GNSS_TX_TO_MODULE renamed LF_DIN_3V3
- net LF_DIN_3V3: now also U21.5 (Pin_5)
- net GPIO38 renamed PAIR_N
- net PAIR_N: now also R509.1, SW6.1
- net GPIO9 renamed BOARD_TEMP_HDR
- net GPIO9_MCU renamed BOARD_TEMP_ADC
- net BOARD_TEMP_ADC: now also R736.2, RT701.1
- net RGB_DOUT4: no longer names the net of LED4.2 (DOUT)
- new net LF_ANT_A: C505.2, J3.1 (Pin_1), R503.1
- new net LF_CEXT: C503.1, U4.12 (CEXT)
- new net LF_CLK_4M: U4.6 (XTAL1), Y501.3 (Pin_3)
- new net LF_DIN_5V: U21.6 (Pin_6), U4.9 (DIN)
- new net LF_DOUT_5V: U22.2, U4.10 (DOUT)
- new net LF_RX: C509.1, R504.2, U4.14 (RX)
- new net LF_SCLK_5V: U21.3 (Pin_3), U4.8 (SCLK)
- new net LF_TX1: C505.1, U4.4 (TX1)
- new net LF_TX2: C506.2, C507.2, C508.2, U4.2 (TX2)
- new net USER_BUTTON_SELECT_N: R607.1, SW7.1, U9.11 (P07)
- no-connect marks 41 -> 48
Other:
- note added: "05 LF RFID / SECURITY / MICROSD"
- note removed: "05 GNSS / ANTENNA / MICROSD"

Commit message: Save shared-SPI LF and plane-fanout checkpoint
Parts:
- removed U22: SN74LVC1G17DBVR LF 5V-TO-3V3, Package_TO_SOT_SMD:SOT-23-5_HandSoldering, symbol 74xGxx:74LVC1G17
- added U22: SN74LVC1G126DBVR LF 5V-TO-3V3 TRI-STATE, Package_TO_SOT_SMD:SOT-23-5_HandSoldering, symbol 74xGxx:74LVC1G126
- C515: value 100nF AHCT supply -> 100nF LV-AT supply
- U21: value SN74AHCT125PWR LF 3V3-TO-5V -> SN74LV125ATPWR LF/SPI 3V3-TO-5V IOFF; LCSC C36365 -> C2675655; MPN SN74AHCT125PWR -> SN74LV125ATPWR
Connections:
- net +3V3: now also U22.5 (VCC)
- net GND: now also U22.3 (GND)
- net LF_DIN_5V: now also U21.3 (Pin_3); no longer U21.6 (Pin_6)
- net LF_DOUT_5V: now also U22.2
- net LF_RFID_EN: now also U22.1
- net LF_SCLK_5V: now also U21.6 (Pin_6); no longer U21.3 (Pin_3)
- net SPI_MISO: now also U22.4
- net SPI_MOSI: now also U21.2 (Pin_2)
- net SPI_SCK: now also U21.5 (Pin_5)
- net LF_DIN_3V3: no longer names the net of U1.28 (IO35)
- net LF_DIN_3V3: no longer U21.5 (Pin_5)
- net LF_DOUT_3V3: no longer names the net of U1.23 (IO21)
- net LF_SCLK_3V3: no longer names the net of U1.11 (IO18)
- net LF_SCLK_3V3: no longer U21.2 (Pin_2)
- no-connect marks 48 -> 50

Commit message: Save PCBA routing optimization checkpoint
Parts:
- added R129: 0R SPI CROSSOVER, Resistor_SMD:R_0805_2012Metric, symbol Device:R
Connections:
- net GND: now also U21.10 (Pin_10), U21.13 (Pin_13), U21.2 (Pin_2); no longer U21.12 (Pin_12)
- net LF_5V: no longer U21.10 (Pin_10), U21.13 (Pin_13)
- net LF_DIN_5V: now also U21.11 (Pin_11); no longer U21.3 (Pin_3)
- net SPI_MOSI: now also U21.12 (Pin_12), R129.2; no longer R402.1, U21.2 (Pin_2)
- new net SPI_MOSI_JMP: R129.1, R402.1

Commit message: Checkpoint zero-open routing and cleanup tooling
Parts:
- removed C610, C611: 1uF X7R, Capacitor_SMD:C_0805_2012Metric, symbol Device:C
- removed C612, C616: 100nF X7R, Capacitor_SMD:C_0805_2012Metric, symbol Device:C
- removed C613, C615: 4.7uF X5R, Capacitor_SMD:C_0805_2012Metric, symbol Device:C
- removed C614: 2.2uF X7R, Capacitor_SMD:C_0805_2012Metric, symbol Device:C
- removed J8: ER-OLED0.42-1W 72x40 SSD1306B, PocketLab_Custom:EastRising_ER-OLED0.42-1W_SolderFPC, symbol Connector_Generic:Conn_01x16
- added SW8: AUX CONFIG, Button_Switch_SMD:SW_SPST_CK_KXT3, symbol Switch:SW_Push
- A1, J3, J5: now left out of the parts list
- C101: LCSC (none) -> C5565742; MPN (none) -> C0805C472KDRAC7800; Manufacturer (none) -> KEMET
- C102, C106, C107, C118, C120, C121, C122, C203, C301, C302, C304, C305, C314, C316, C317, C401, C501, C503, C504, C510, C513, C515, C516, C517, C601, C603, C604, C605, C606, C608, C609, C701, C706, C707: footprint Capacitor_SMD:C_0805_2012Metric -> Capacitor_SMD:C_0402_1005Metric; LCSC (none) -> C1525; MPN (none) -> CL05B104KO5NNNC; Manufacturer (none) -> Samsung Electro-Mechanics
- C103, C105, C303, C315, C402, C602: footprint Capacitor_SMD:C_0805_2012Metric -> Capacitor_SMD:C_0603_1608Metric; LCSC (none) -> C19666; MPN (none) -> CL10A475KO8NNNC; Manufacturer (none) -> Samsung Electro-Mechanics
- C104, C110, C111, C112, C115, C116: LCSC (none) -> C380336; MPN (none) -> TCC0805X5R226K100FT; Manufacturer (none) -> CCTC
- C108, C109, C114, C117, C119, C502: LCSC (none) -> C15850; MPN (none) -> CL21A106KAYNNNE; Manufacturer (none) -> Samsung Electro-Mechanics
- C113, C308, C309, C508: LCSC (none) -> C27675; MPN (none) -> CL10C221JB8NNNC; Manufacturer (none) -> Samsung Electro-Mechanics
- C123, C124: footprint Capacitor_SMD:C_0603_1608Metric -> Capacitor_SMD:C_0805_2012Metric; LCSC (none) -> C15850; MPN (none) -> CL21A106KAYNNNE; Manufacturer (none) -> Samsung Electro-Mechanics
- C201: footprint Capacitor_SMD:C_0805_2012Metric -> Capacitor_SMD:C_0402_1005Metric; LCSC (none) -> C52923; MPN (none) -> CL05A105KA5NQNC; Manufacturer (none) -> Samsung Electro-Mechanics
- C202, C313, C511: footprint Capacitor_SMD:C_0805_2012Metric -> Capacitor_SMD:C_0603_1608Metric; LCSC (none) -> C19702; MPN (none) -> CL10A106KP8NNNC; Manufacturer (none) -> Samsung Electro-Mechanics
- C306, C307: LCSC (none) -> C1653; MPN (none) -> CL10C220JB8NNNC; Manufacturer (none) -> Samsung Electro-Mechanics
- C318: LCSC (none) -> C163508; MPN (none) -> CL10C102JB8NNNC; Manufacturer (none) -> Samsung Electro-Mechanics
- C403, C404: footprint Capacitor_SMD:C_0805_2012Metric -> Capacitor_SMD:C_0603_1608Metric
- C505: footprint Capacitor_SMD:C_0805_2012Metric -> Capacitor_SMD:C_1206_3216Metric; LCSC (none) -> C46348; MPN (none) -> 1206CG104J500NT; Manufacturer (none) -> FH
- C506: LCSC (none) -> C307553; MPN (none) -> CL21C392JBFNNNE; Manufacturer (none) -> Samsung Electro-Mechanics
- C507: LCSC (none) -> C14858; MPN (none) -> CL10C101JB8NNNC; Manufacturer (none) -> Samsung Electro-Mechanics
- C509: LCSC (none) -> C1634; MPN (none) -> CL10C100JB8NNNC; Manufacturer (none) -> Samsung Electro-Mechanics
- C512: footprint Capacitor_SMD:C_1210_3225Metric -> Capacitor_SMD:C_1206_3216Metric; LCSC (none) -> C110047; MPN GRM32ER60J476ME20L -> CC1206MKX5R5BB476; Manufacturer Murata -> Yageo
- C607, C617: LCSC (none) -> C7393980; MPN (none) -> TCC1206X5R226K100HT; Manufacturer (none) -> CCTC
- C702, C703, C704, C705: footprint Capacitor_SMD:C_0603_1608Metric -> Capacitor_SMD:C_0402_1005Metric; LCSC (none) -> C1525; MPN (none) -> CL05B104KO5NNNC; Manufacturer (none) -> Samsung Electro-Mechanics
- D1, D2, D3: value TSAL6200 940nm -> VSMY14940 940nm side-view; footprint PocketLab_Custom:TSAL6200_LayFlat_Inboard -> PocketLab_Custom:LED_Vishay_VSMY14940_SideView; Assembly MANUAL_EDGE_BEND -> (none); LCSC C55528 -> C511069; MPN TSAL6200 -> VSMY14940
- D101: LCSC (none) -> C151296
- F1: LCSC (none) -> C207036; MPN (none) -> 1206L075/13.2WR; Manufacturer (none) -> Littelfuse
- J2: LCSC (none) -> C585350; MPN (none) -> 104031-0811; Manufacturer (none) -> Molex
- J4: LCSC (none) -> C295747; MPN S2B-PH-SM4-TB -> S2B-PH-SM4-TB(LF)(SN)
- L301, L302: LCSC (none) -> C304279; MPN (none) -> FHW0805UFR56JST; Manufacturer (none) -> FH
- L6: value 1.5uH XFL4020-152ME -> 1.5uH 5.2A SMHT4020; footprint PocketLab_Custom:Coilcraft_XFL4020 -> PocketLab_Custom:ShunXiangNuo_SMHT4020; LCSC (none) -> C46469583; MPN (none) -> SMHT4020-1R5MT; Manufacturer (none) -> Shun Xiang Nuo
- L7: value 1uH HBME042A -> 1uH 4.15A SLW4030S; footprint PocketLab_Custom:Cyntec_HBME042A-1R0MS -> PocketLab_Custom:Sunltech_SLW4030S; LCSC (none) -> C206354; MPN (none) -> SLW4030S1R0NST; Manufacturer (none) -> Sunltech
- Q2, Q3: LCSC (none) -> C2861720
- R101, R102: footprint Resistor_SMD:R_0805_2012Metric -> Resistor_SMD:R_0402_1005Metric; LCSC (none) -> C25905; MPN (none) -> 0402WGF5101TCE; Manufacturer (none) -> UNI-ROYAL
- R103: footprint Resistor_SMD:R_0805_2012Metric -> Resistor_SMD:R_0402_1005Metric; LCSC (none) -> C26083; MPN (none) -> 0402WGF1004TCE; Manufacturer (none) -> UNI-ROYAL
- R104: footprint Resistor_SMD:R_0805_2012Metric -> Resistor_SMD:R_0402_1005Metric; LCSC (none) -> C25104; MPN (none) -> 0402WGF3300TCE; Manufacturer (none) -> UNI-ROYAL
- R105: LCSC (none) -> C17520; MPN (none) -> 0805W8F2201T5E; Manufacturer (none) -> UNI-ROYAL
- R106, R107: footprint Resistor_SMD:R_0805_2012Metric -> Resistor_SMD:R_0402_1005Metric; LCSC (none) -> C270595; MPN (none) -> 0402WGF5104TCE; Manufacturer (none) -> UNI-ROYAL
- R108, R119: LCSC (none) -> C17414; MPN (none) -> 0805W8F1002T5E; Manufacturer (none) -> UNI-ROYAL
- R109, R110, R115, R121, R122, R124, R126, R127, R128, R406, R506, R603: footprint Resistor_SMD:R_0805_2012Metric -> Resistor_SMD:R_0402_1005Metric; LCSC (none) -> C25741; MPN (none) -> 0402WGF1003TCE; Manufacturer (none) -> UNI-ROYAL
- R111: footprint Resistor_SMD:R_0805_2012Metric -> Resistor_SMD:R_0402_1005Metric; LCSC (none) -> C22065; MPN (none) -> 0402WGF3481TCE; Manufacturer (none) -> UNI-ROYAL
- R112: footprint Resistor_SMD:R_0805_2012Metric -> Resistor_SMD:R_0402_1005Metric; LCSC (none) -> C25889; MPN (none) -> 0402WGF3011TCE; Manufacturer (none) -> UNI-ROYAL
- R113: footprint Resistor_SMD:R_0805_2012Metric -> Resistor_SMD:R_0402_1005Metric; LCSC (none) -> C113478; MPN (none) -> 0402WGF1781TCE; Manufacturer (none) -> UNI-ROYAL
- R114: footprint Resistor_SMD:R_0805_2012Metric -> Resistor_SMD:R_0402_1005Metric; LCSC (none) -> C11537; MPN (none) -> 0402WGF6812TCE; Manufacturer (none) -> UNI-ROYAL
- R116, R125, R203, R204, R301, R302, R509, R519, R703: footprint Resistor_SMD:R_0805_2012Metric -> Resistor_SMD:R_0402_1005Metric; LCSC (none) -> C25744; MPN (none) -> 0402WGF1002TCE; Manufacturer (none) -> UNI-ROYAL
- R117: footprint Resistor_SMD:R_0805_2012Metric -> Resistor_SMD:R_0402_1005Metric; LCSC (none) -> C25790; MPN (none) -> 0402WGF4703TCE; Manufacturer (none) -> UNI-ROYAL
- R118, R504: footprint Resistor_SMD:R_0805_2012Metric -> Resistor_SMD:R_0402_1005Metric; LCSC (none) -> C25755; MPN (none) -> 0402WGF1503TCE; Manufacturer (none) -> UNI-ROYAL
- R120: footprint Resistor_SMD:R_0805_2012Metric -> Resistor_SMD:R_0402_1005Metric; LCSC (none) -> C27016; MPN (none) -> 0402WGF7323TCE; Manufacturer (none) -> UNI-ROYAL
- R123: footprint Resistor_SMD:R_0805_2012Metric -> Resistor_SMD:R_0402_1005Metric; LCSC (none) -> C25911; MPN (none) -> 0402WGF6042TCE; Manufacturer (none) -> UNI-ROYAL
- R201, R202: LCSC (none) -> C17561; MPN (none) -> 0805W8F220JT5E; Manufacturer (none) -> UNI-ROYAL
- R303, R304, R405: footprint Resistor_SMD:R_0805_2012Metric -> Resistor_SMD:R_0603_1608Metric; LCSC (none) -> C21189; MPN (none) -> 0603WAF0000T5E; Manufacturer (none) -> UNI-ROYAL
- R305: footprint Resistor_SMD:R_0805_2012Metric -> Resistor_SMD:R_0603_1608Metric; LCSC (none) -> C13167; MPN (none) -> 0603WAF2701T5E; Manufacturer (none) -> UNI-ROYAL
- R306: footprint Resistor_SMD:R_0805_2012Metric -> Resistor_SMD:R_0603_1608Metric; LCSC (none) -> C21190; MPN (none) -> 0603WAF1001T5E; Manufacturer (none) -> UNI-ROYAL
- R401, R402, R403, R404, R510, R511, R512, R513: footprint Resistor_SMD:R_0805_2012Metric -> Resistor_SMD:R_0402_1005Metric; LCSC (none) -> C25092; MPN (none) -> 0402WGF220JTCE; Manufacturer (none) -> UNI-ROYAL
- R501, R602, R604: footprint Resistor_SMD:R_0805_2012Metric -> Resistor_SMD:R_0402_1005Metric; LCSC (none) -> C25076; MPN (none) -> 0402WGF1000TCE; Manufacturer (none) -> UNI-ROYAL
- R502: LCSC (none) -> C474213; MPN (none) -> 1210W2F470JT5E; Manufacturer (none) -> UNI-ROYAL
- R503: footprint Resistor_SMD:R_0805_2012Metric -> Resistor_SMD:R_0402_1005Metric; LCSC (none) -> C11702; MPN (none) -> 0402WGF1001TCE; Manufacturer (none) -> UNI-ROYAL
- R514, R515, R516, R517, R518: footprint Resistor_SMD:R_0805_2012Metric -> Resistor_SMD:R_0402_1005Metric; LCSC (none) -> C25792; MPN (none) -> 0402WGF4702TCE; Manufacturer (none) -> UNI-ROYAL
- R601, R610, R611: value 39R 0.5W pulse-rated -> 68R 0.25W anti-surge; footprint Resistor_SMD:R_1210_3225Metric -> Resistor_SMD:R_0603_1608Metric; LCSC (none) -> C966162; MPN (none) -> AS03W4J0680T5E; Manufacturer (none) -> UNI-ROYAL
- R605: footprint Resistor_SMD:R_0603_1608Metric -> Resistor_SMD:R_0402_1005Metric; LCSC (none) -> C25131; MPN (none) -> 0402WGF680JTCE; Manufacturer (none) -> UNI-ROYAL
- R606, R710, R711, R712, R713, R714, R715, R716, R717, R718, R719, R720, R721, R730, R731, R732, R733, R734: footprint Resistor_SMD:R_0603_1608Metric -> Resistor_SMD:R_0402_1005Metric; LCSC (none) -> C25076; MPN (none) -> 0402WGF1000TCE; Manufacturer (none) -> UNI-ROYAL
- R607, R608, R609: footprint Resistor_SMD:R_0603_1608Metric -> Resistor_SMD:R_0402_1005Metric; LCSC (none) -> C25744; MPN (none) -> 0402WGF1002TCE; Manufacturer (none) -> UNI-ROYAL
- R701: LCSC (none) -> C26010; MPN (none) -> 0805W8F3301T5E; Manufacturer (none) -> UNI-ROYAL
- R702: footprint Resistor_SMD:R_0805_2012Metric -> Resistor_SMD:R_0402_1005Metric; LCSC (none) -> C25890; MPN (none) -> 0402WGF3301TCE; Manufacturer (none) -> UNI-ROYAL
- R722, R723, R724, R725, R726, R727, R728, R729: footprint Resistor_SMD:R_0603_1608Metric -> Resistor_SMD:R_0402_1005Metric; LCSC (none) -> C25091; MPN (none) -> 0402WGF2200TCE; Manufacturer (none) -> UNI-ROYAL
- R735: LCSC (none) -> C149504; MPN (none) -> 0805W8F1003T5E; Manufacturer (none) -> UNI-ROYAL
- R736: footprint Resistor_SMD:R_0603_1608Metric -> Resistor_SMD:R_0402_1005Metric; LCSC C25804 -> C25744; MPN 0603WAF1002T5E -> 0402WGF1002TCE
- SW1, SW2, SW3, SW4, SW6, SW7: footprint Button_Switch_SMD:SW_Push_1P1T_NO_CK_KMR2 -> PocketLab_Custom:SW_HYP_1TS015A_3.0x2.0mm; LCSC C72443 -> C256104; MPN KMR221GLFS -> 1TS015A-1600-0600-CT; Manufacturer C&K -> HYP
- U13: LCSC (none) -> C7365598
- U14: LCSC (none) -> C183096
- U15: LCSC (none) -> C55266
- U16: LCSC (none) -> C435848
- U18: LCSC (none) -> C783615
- U19, U24, U25: LCSC (none) -> C604719
- U22: footprint Package_TO_SOT_SMD:SOT-23-5_HandSoldering -> Package_TO_SOT_SMD:SOT-23-5
- Y301: LCSC (none) -> C124317; MPN (none) -> XXDBBCNANF-27.12M; Manufacturer (none) -> TAITIEN
- Y501: footprint Oscillator:Oscillator_SMD_EuroQuartz_XO32-4Pin_3.2x2.5mm_RotB_HandSoldering -> Oscillator:Oscillator_SMD_EuroQuartz_XO32-4Pin_3.2x2.5mm_RotB
- Y701: LCSC (none) -> C276424
Connections:
- net GND: now also SW8.2
- net USER_BUTTON_AUX_N: now reaches U1.23 (IO21)
- net USER_BUTTON_AUX_N: now also SW8.1
- no-connect marks 50 -> 49
Other:
- note added: "06 IR / RGB / BUTTONS"
- note removed: "06 IR / RGB / BUTTONS / OLED"
