File: hardware/PocketLab-Card.kicad_pcb (KiCad board)
At the start: 4 copper layers, 85.6 x 54 mm, 267 parts, among them J1 USB-C DATA/POWER, J2 microSD, J3 EXTERNAL 400uH LF COIL, J4 PROTECTED 1S LiPo 3.7V, J5 30-PIN 2.54mm DUPONT GRID, J8 ER-OLED0.42-1W 72x40 SSD1306B, Q1 AO3400A IR DRIVER, Q2 CSD16406Q3 DISCHARGE, Q3 CSD16406Q3 CHARGE, SW1 RESET, SW2 BOOT, SW3 UP, SW4 DOWN, SW5 MAIN POWER OFF / ON, SW6 PAIR, SW7 SELECT, U1 ESP32-S3-WROOM-1-N8R2, U10 BMI270 (FULL OPTION), U11 BMP390 (FULL OPTION), U12 PCF8563T, U13 TSOP75338WTR 38kHz, U14 BQ29700DSE, U15 TPS2553DBVR 500mA LIMIT, U16 USBLC6-4SC6Y, U17 TPS22919DCKR LF 5V LOAD SWITCH, U18 TCA9534PWR INTERNAL CONTROL, U19 SRV05-4MR6T1G SD ESD, U2 PN5321A3HN/C106, U20 SN74AHCT1G126DBVR RGB LEVEL S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, U21 SN74LV125ATPWR LF/SPI 3V3-TO-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, U22 SN74LVC1G126DBVR LF 5V-TO-3V3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, U23 ATECC608C-SSHDA-T, U24 SRV05-4MR6T1G J5 BUS ESD, U25 SRV05-4MR6T1G J5 SPI ESD, U3 E07-900MM10S 855-925MHz, U4 HTRC11001T/03EE,11 125kHz, U5 BQ24074RGTR, U6 TPS63070RNMR 3V3, U7 TPS61023DRLR 5V BOOST, U8 MAX17048G+T10, U9 TCA9535PWR, Y301 27.12MHz crystal (pins 2/4 sh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, Y501 4MHz 5V CMOS OSCILLATOR, Y701 32.768kHz CL=7pF

Commit message: Route protected SPI MISO header branch
Routing:
- net /SPI_MISO_HDR: track 0.00 -> 17.5 mm, vias 0 -> 2
Changed lines of the file:
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@@
+	)
+	(segment
+		(start 91.3 66.4)
+		(end 92.15 66.75)
+		(width 0.15)
+		(locked yes)
+		(layer "F.Cu")
+		(net "/SPI_MISO_HDR")
+	)
+	(segment
+		(start 89.85 66.4)
+		(end 91.3 66.4)
+		(width 0.15)
+		(locked yes)
+		(layer "F.Cu")
+		(net "/SPI_MISO_HDR")
+	)
+	(segment
+		(start 89.85 65.575)
+		(end 89.85 66.4)
+		(width 0.15)
+		(locked yes)
+		(layer "F.Cu")
+		(net "/SPI_MISO_HDR")
+	)
+	(via
+		(at 92.15 66.75)
+		(size 0.45)
+		(drill 0.2)
+		(layers "F.Cu" "B.Cu")
+		(locked yes)
+		(net "/SPI_MISO_HDR")
+	)
+	(via
+		(at 82 59.2)
+		(size 0.45)
+		(drill 0.2)
+		(layers "F.Cu" "B.Cu")
+		(locked yes)
+		(net "/SPI_MISO_HDR")
+	)
+	(segment
+		(start 84.3 58.85)
+		(end 85.1 59.65)
+		(width 0.15)
+		(locked yes)
+		(layer "In2.Cu")
+		(net "/SPI_MISO_HDR")
+	)
+	(segment
+		(start 85.1 61.4)
+		(end 86 62.8)
+		(width 0.15)
+		(locked yes)
+		(layer "In2.Cu")
+		(net "/SPI_MISO_HDR")
+	)
+	(segment
+		(start 86 62.8)
+		(end 88 63.8)
+		(width 0.15)
+		(locked yes)
+		(layer "In2.Cu")
+		(net "/SPI_MISO_HDR")
+	)
+	(segment
+		(start 82.5 58.85)
+		(end 84.3 58.85)
+		(width 0.15)
+		(locked yes)
+		(layer "In2.Cu")
+		(net "/SPI_MISO_HDR")
+	)
+	(segment
+		(start 88 63.8)
+		(end 89.25 65)
+		(width 0.15)
+		(locked yes)
+		(layer "In2.Cu")
+		(net "/SPI_MISO_HDR")
+	)
+	(segment
+		(start 82 59.2)
+		(end 82.5 58.85)
+		(width 0.15)
+		(locked yes)
+		(layer "In2.Cu")
+		(net "/SPI_MISO_HDR")
+	)
+	(segment
+		(start 89.25 65)
+		(end 92.15 66.75)
+		(width 0.15)
+		(locked yes)
+		(layer "In2.Cu")
+		(net "/SPI_MISO_HDR")
+	)
+	(segment
+		(start 85.1 59.65)
+		(end 85.1 61.4)
+		(width 0.15)
+		(locked yes)
+		(layer "In2.Cu")
+		(net "/SPI_MISO_HDR")
 	)
 	(segment
