File: hardware/PocketLab-Card.kicad_pcb (KiCad board)
At the start: 4 copper layers, 85.6 x 54 mm, 267 parts, among them J1 USB-C DATA/POWER, J2 microSD, J3 EXTERNAL 400uH LF COIL, J4 PROTECTED 1S LiPo 3.7V, J5 30-PIN 2.54mm DUPONT GRID, J8 ER-OLED0.42-1W 72x40 SSD1306B, Q1 AO3400A IR DRIVER, Q2 CSD16406Q3 DISCHARGE, Q3 CSD16406Q3 CHARGE, SW1 RESET, SW2 BOOT, SW3 UP, SW4 DOWN, SW5 MAIN POWER OFF / ON, SW6 PAIR, SW7 SELECT, U1 ESP32-S3-WROOM-1-N8R2, U10 BMI270 (FULL OPTION), U11 BMP390 (FULL OPTION), U12 PCF8563T, U13 TSOP75338WTR 38kHz, U14 BQ29700DSE, U15 TPS2553DBVR 500mA LIMIT, U16 USBLC6-4SC6Y, U17 TPS22919DCKR LF 5V LOAD SWITCH, U18 TCA9534PWR INTERNAL CONTROL, U19 SRV05-4MR6T1G SD ESD, U2 PN5321A3HN/C106, U20 SN74AHCT1G126DBVR RGB LEVEL S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, U21 SN74LV125ATPWR LF/SPI 3V3-TO-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, U22 SN74LVC1G126DBVR LF 5V-TO-3V3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, U23 ATECC608C-SSHDA-T, U24 SRV05-4MR6T1G J5 BUS ESD, U25 SRV05-4MR6T1G J5 SPI ESD, U3 E07-900MM10S 855-925MHz, U4 HTRC11001T/03EE,11 125kHz, U5 BQ24074RGTR, U6 TPS63070RNMR 3V3, U7 TPS61023DRLR 5V BOOST, U8 MAX17048G+T10, U9 TCA9535PWR, Y301 27.12MHz crystal (pins 2/4 sh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, Y501 4MHz 5V CMOS OSCILLATOR, Y701 32.768kHz CL=7pF

Commit message: Checkpoint active PCB routing and tooling
Parts:
- R610, TP107: moved to B.Cu
- moved R610 48.3 mm to (28.8, 54.6), turned to 180 degrees
- moved TP107 44.9 mm to (84.8, 52.0), turned to 180 degrees
Routing:
- net /BOARD_TEMP_ADC: track 2.68 -> 127.8 mm, vias 0 -> 4
- net /GPIO47: track 0.00 -> 99.4 mm, vias 0 -> 1
- net /NFC_RX: track 0.00 -> 83.3 mm, vias 0 -> 3
- net /GPIO48: track 0.00 -> 71.8 mm, vias 0 -> 1
- net /PAIR_N: track 13.7 -> 78.3 mm, vias 2 -> 5
- net /NFC_DVDD: track 4.22 -> 63.6 mm, vias 0 -> 9
- net /NFC_RX_AC: track 0.00 -> 58.6 mm, vias 0 -> 2
- net /IR_RX: track 0.00 -> 44.8 mm, vias 0 -> 2
- net /IR_LED_K: track 16.4 -> 58.0 mm, vias 0 -> 2
- net /IOEXP_INT_N: track 3.40 -> 42.8 mm, vias 0 -> 6
- net /NFC_TX1_F: track 0.00 -> 34.5 mm, vias 0 -> 3
- net /I2C_SCL: track 8.41 -> 36.0 mm, vias 3 -> 11
- net /SPI_MISO: track 33.9 -> 59.7 mm, vias 4 -> 5
- net /GND: track 392.6 -> 412.5 mm, vias 133 -> 145
- net /SPI_SCK: track 42.6 -> 61.4 mm, vias 2 -> 5
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
Commit message: Checkpoint zero-open routing and cleanup tooling
Routing:
- net /+5V_RAW: track 70.2 -> 118.0 mm, vias 19 -> 28
- net /BQ_EN2: track 0.00 -> 46.6 mm, vias 0 -> 2
- net /CHARGER_CHG_N: track 0.00 -> 32.1 mm, vias 0 -> 2
- net /EX7_INT: track 0.00 -> 28.4 mm, vias 0 -> 2
- net /EX6_INT: track 0.00 -> 23.8 mm, vias 0 -> 2
- net /I2C_SCL: track 36.0 -> 59.5 mm, vias 11 -> 14
- net /CHG_TMR: track 0.00 -> 22.9 mm, vias 0 -> 2
- net /CHARGER_PGOOD_N: track 0.00 -> 20.3 mm, vias 0 -> 2
- net /NFC_VMID: track 0.00 -> 16.0 mm
- net /I2C_SDA: track 32.1 -> 42.2 mm, vias 7 -> 9
- net /CHG_ITERM: track 0.00 -> 9.82 mm, vias 0 -> 2
- net /BOOST5_EN: track 0.00 -> 8.18 mm, vias 0 -> 2
- net /NFC_TX2: track 0.00 -> 7.23 mm, vias 0 -> 4
- net /+3V3: track 296.8 -> 301.1 mm
- net /NFC_I0: track 17.9 -> 22.2 mm
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- added copper zone on B.Cu, net /+3V3
