File: hardware/PocketLab-Card-routing-working.kicad_pcb (KiCad board)
At the start: 4 copper layers, 85.6 x 54 mm, 260 parts, among them J1 USB-C DATA/POWER, J2 microSD, J3 EXTERNAL 400uH LF COIL, J4 PROTECTED 1S LiPo 3.7V, J5 30-PIN 2.54mm DUPONT GRID, Q1 AO3400A IR DRIVER, Q2 CSD16406Q3 DISCHARGE, Q3 CSD16406Q3 CHARGE, SW1 RESET, SW2 BOOT, SW3 UP, SW4 DOWN, SW5 MAIN POWER OFF / ON, SW6 PAIR, SW7 SELECT, SW8 AUX CONFIG, U1 ESP32-S3-WROOM-1-N8R2, U10 BMI270 (FULL OPTION), U11 BMP390 (FULL OPTION), U12 PCF8563T, U13 TSOP75338WTR 38kHz, U14 BQ29700DSE, U15 TPS2553DBVR 500mA LIMIT, U16 USBLC6-4SC6Y, U17 TPS22919DCKR LF 5V LOAD SWITCH, U18 TCA9534PWR INTERNAL CONTROL, U19 SRV05-4MR6T1G SD ESD, U2 PN5321A3HN/C106, U20 SN74AHCT1G126DBVR RGB LEVEL S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, U21 SN74LV125ATPWR LF/SPI 3V3-TO-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, U22 SN74LVC1G126DBVR LF 5V-TO-3V3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, U23 ATECC608C-SSHDA-T, U24 SRV05-4MR6T1G J5 BUS ESD, U25 SRV05-4MR6T1G J5 SPI ESD, U3 E07-900MM10S 855-925MHz, U4 HTRC11001T/03EE,11 125kHz, U5 BQ24074RGTR, U6 TPS63070RNMR 3V3, U7 TPS61023DRLR 5V BOOST, U8 MAX17048G+T10, U9 TCA9535PWR, Y301 27.12MHz crystal (pins 2/4 sh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, Y501 4MHz 5V CMOS OSCILLATOR, Y701 32.768kHz CL=7pF

Commit message: Remove copper sliver and GPIO8 edge faults
Routing:
- net /GPIO8_MCU: track 102.0 -> 100.8 mm
- net /GND: track 760.2 -> 760.8 mm
Changed lines of the file:
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@@
 	)
 	(segment
+		(start 49.96 54.8361)
+		(end 49.3 54.95)
+		(width 0.6)
+		(layer "In2.Cu")
+		(net "/GND")
+	)
+	(segment
 		(start 69.0506 63.3878)
 		(end 70.1131 63.3878)
@@
 	)
 	(segment
-		(start 21.2 20.75)
-		(end 21.2 52.8)
+		(start 23.2 20.75)
+		(end 22.2 21.5)
 		(width 0.15)
 		(locked yes)
@@
 	)
 	(segment
-		(start 24.925 20.75)
-		(end 21.2 20.75)
+		(start 21.2 23.2)
+		(end 21.2 52.8)
 		(width 0.15)
 		(locked yes)
@@
 		(width 0.15)
 		(locked yes)
+		(layer "In2.Cu")
+		(net "/GPIO8_MCU")
+	)
+	(segment
+		(start 24.925 20.75)
+		(end 23.2 20.75)
+		(width 0.15)
+		(locked yes)
+		(layer "In2.Cu")
+		(net "/GPIO8_MCU")
+	)
+	(segment
+		(start 22.2 21.5)
+		(end 21.2 23.2)
+		(width 0.15)
+		(locked yes)

Commit message: Merge redundant routing vias
Routing:
- net /SD_SCK: track 31.0 -> 31.1 mm, vias 3 -> 2
- net /NFC_SVDD: track 6.83 -> 6.80 mm, vias 2 -> 1
- net /BAT_SENSE: vias 6 -> 5
Changed lines of the file:
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@@
 	)
 	(segment
-		(start 68.695 39.525)
+		(start 68.45 39.4625)
 		(end 69.495 40.325)
 		(width 0.15)
@@
 		(net "/NFC_SVDD")
 	)
-	(via
-		(at 68.695 39.525)
-		(size 0.5)
-		(drill 0.3)
-		(layers "F.Cu" "B.Cu")
-		(net "/NFC_SVDD")
-	)
-	(segment
-		(start 68.45 39.4625)
-		(end 68.695 39.525)
-		(width 0.15)
-		(layer "B.Cu")
-		(net "/NFC_SVDD")
-	)
 	(segment
 		(start 63.75 38.4625)
@@
 		(net "/SD_SCK")
 	)
-	(via
-		(at 103.1 36.2)
-		(size 0.45)
-		(drill 0.2)
-		(layers "F.Cu" "B.Cu")
-		(locked yes)
-		(tenting
-			(front yes)
-			(back yes)
-		)
-		(net "/SD_SCK")
-	)
 	(segment
 		(start 104.55 37.705)
@@
 	(segment
 		(start 103.55 37.305)
-		(end 103.1 36.2)
+		(end 102.95 36.105)
 		(width 0.15)
 		(locked yes)
@@
 	(segment
 		(start 82.2 48.7125)
-		(end 103.1 36.2)
+		(end 102.95 36.105)
 		(width 0.15)
 		(locked yes)
@@
 	)
 	(segment
-		(start 85 64.45)
-		(end 84.825 64.5)
-		(width 0.15)
-		(layer "F.Cu")
-		(net "/BAT_SENSE")
-	)
-	(segment
 		(start 87.675 64)
 		(end 87.425 64.75)
@@
 		(net "/BAT_SENSE")
 	)
-	(via
-		(at 85 64.45)
-		(size 0.5)
-		(drill 0.3)
-		(layers "F.Cu" "B.Cu")
-		(net "/BAT_SENSE")
-	)
 	(segment
 		(start 87.925 67)
@@
 	(segment
 		(start 85.6 64.45)
-		(end 85 64.45)
+		(end 84.825 64.5)
 		(width 0.15)
 		(layer "B.Cu")

Commit message: Make USB connector P join via-free
Routing:
- net /USB_CONN_P: vias 2 -> 0
Changed lines of the file:
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@@
 	)
 	(segment
-		(start 97.155 50.75)
+		(start 96.8 50.4625)
 		(end 97.355 50.95)
 		(width 0.15)
@@
 		(net "/USB_CONN_P")
 	)
-	(via
-		(at 96.8 50.4625)
-		(size 0.5)
-		(drill 0.3)
-		(layers "F.Cu" "B.Cu")
-		(net "/USB_CONN_P")
-	)
-	(via
-		(at 97.155 50.75)
-		(size 0.5)
-		(drill 0.3)
-		(layers "F.Cu" "B.Cu")
-		(net "/USB_CONN_P")
-	)
-	(segment
-		(start 96.8 50.4625)
-		(end 97.155 50.75)
-		(width 0.15)
-		(layer "B.Cu")
-		(net "/USB_CONN_P")
-	)

Commit message: Save conventional via cleanup checkpoint
Routing:
- net /CHG_TS: track 53.0 -> 61.0 mm
- net /IR_TX: track 42.7 -> 43.8 mm
- net /NFC_OSCOUT: track 6.17 -> 6.08 mm, vias 2 -> 1
Changed lines of the file:
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@@
 	)
 	(segment
-		(start 86.9 50.15)
+		(start 86.75 50.15)
 		(end 87.3625 50.15)
 		(width 0.2)
@@
 	)
 	(via
-		(at 59.39 48.5361)
+		(at 59.2082 48.6602)
 		(size 0.5)
 		(drill 0.3)
@@
 	)
 	(via
-		(at 86.9 50.15)
+		(at 86.75 50.15)
 		(size 0.5)
 		(drill 0.3)
@@
 	(segment
 		(start 86.9 49.55)
-		(end 86.9 50.15)
+		(end 86.75 50.15)
 		(width 0.2)
 		(layer "B.Cu")
@@
 	(segment
 		(start 59.85 49.8)
-		(end 59.39 48.5361)
+		(end 59.2082 48.6602)
 		(width 0.2)
 		(layer "B.Cu")
@@
 	)
 	(segment
-		(start 63.25 40)
+		(start 63.6 40.35)
 		(end 63.25 38.9125)
 		(width 0.15)
@@
 	)
 	(via
-		(at 63.25 40)
+		(at 63.6 40.35)
 		(size 0.45)
 		(drill 0.2)
@@
 	(segment
 		(start 62.0625 42.35)
-		(end 63.25 40)
+		(end 63.6 40.35)
 		(width 0.15)
 		(locked yes)
@@
 		(net "/BOOT_N")
 	)
+	(segment
+		(start 66.2 65.7125)
+		(end 65.65 65.7125)
+		(width 0.15)
+		(locked yes)
+		(layer "F.Cu")
+		(net "/IR_TX")
+	)
 	(via
 		(at 101.35 41.46)
@@
 	)
 	(via
-		(at 66.2 65.7125)
+		(at 65.65 65.7125)
 		(size 0.45)
 		(drill 0.2)
@@
 	(segment
 		(start 66.2 65.7125)
+		(end 65.65 65.7125)
+		(width 0.15)
+		(locked yes)
+		(layer "In1.Cu")
+		(net "/IR_TX")
+	)
+	(segment
+		(start 66.2 65.7125)
 		(end 101.35 41.46)
 		(width 0.15)
@@
 	)
 	(segment
-		(start 66.75 47.3375)
+		(start 66.7 47.55)
 		(end 65.75 46.3375)
 		(width 0.15)
@@
 	)
 	(via
-		(at 66.75 47.3375)
-		(size 0.5)
-		(drill 0.3)
-		(layers "F.Cu" "B.Cu")
-		(net "/NFC_OSCOUT")
-	)
-	(via
 		(at 66.7 47.55)
 		(size 0.5)
@@
 		(net "/NFC_OSCOUT")
 	)
-	(segment
-		(start 66.7 47.55)
-		(end 66.75 47.3375)
-		(width 0.15)
-		(layer "B.Cu")
-		(net "/NFC_OSCOUT")
-	)
 	(via
 		(at 65.25 45.5375)
@@
 	)
 	(segment
-		(start 57.27 68)
+		(start 85.645 62)
 		(end 85.645 68)
 		(width 0.15)
@@
 	)
 	(segment
+		(start 57.27 68)
+		(end 65.4 62)
+		(width 0.15)
+		(locked yes)
+		(layer "In2.Cu")
+		(net "/CHG_TS")
+	)
+	(segment
+		(start 65.4 62)
+		(end 85.645 62)
+		(width 0.15)
+		(locked yes)
+		(layer "In2.Cu")
+		(net "/CHG_TS")
+	)
+	(segment
 		(start 57.27 72.08)
 		(end 57.27 68)
@@
 	)
 	(via
-		(at 91.6375 50.75)
+		(at 91.4 50.75)
 		(size 0.45)
 		(drill 0.2)
@@
 	)
 	(segment
+		(start 91.6375 50.75)
+		(end 91.4 50.75)
+		(width 0.15)
+		(layer "B.Cu")
+		(net "/CHG_ITERM")
+	)
+	(segment
 		(start 86.1125 56.2)
-		(end 91.6375 50.75)
+		(end 91.4 50.75)
 		(width 0.15)
 		(locked yes)
