File: hardware/sheets/05_LF_RFID_SD.kicad_sch (KiCad schematic)
At the start: 0 parts

Commit message: Save RFID and critical routing checkpoint
Other:
- title: 05 GNSS SD - CAPTURE TARGET -> 05 LF RFID SECURITY SD - CAPTURE TARGET
Changed lines of the file:
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@@
 	(generator_version "10.0")
 	(paper "A4")
-	(title_block (title "05 GNSS SD - CAPTURE TARGET"))
+	(title_block (title "05 LF RFID SECURITY SD - CAPTURE TARGET"))
 	(sheet_instances (path "/" (page "1")))
 	(embedded_fonts no)
